File: pll.kicad_sch (KiCad schematic)
At the start: 63 parts, among them CN11 UE75-A20-6000T, CN12 U77-A1114-30L1, CN15 731385033, Q6 DMN62D0U-7, T4 TC2-72T+, U11 SY75576LKY, U15 SN74LVC1G02DCK, U3 TI TPS79301DBV

Commit message: Moved to preferred library
Parts:
- C15, C17, C7: symbol Auto_Library_WUT:Samsung Electro-Mechanics CL10A106MO8NQNC -> Preferred_WUT:Samsung Electro-Mechanics CL10A106MO8NQNC
- C157, C159, C35, C9: symbol Auto_Library_WUT:Yageo CC0402KRX7R8BB104 -> Preferred_WUT:Yageo CC0402KRX7R8BB104
- D9: symbol Auto_Library_WUT:Littelfuse AQ3522-01LTG -> Preferred_WUT:Littelfuse AQ3522-01LTG
- FB26, FB27: symbol Auto_Library_WUT:Murata BLM18AG601SN1D -> Preferred_WUT:Murata BLM18AG601SN1D
- LD8: symbol Auto_Library_WUT:Ekinglux_E6C0603VGAC1UDA -> Preferred_WUT:Ekinglux_E6C0603VGAC1UDA
- R100, R101, R105, R106, R110, R111: symbol Auto_Library_WUT:KOA Speer RK73H1ETTP33R0F -> Preferred_WUT:KOA Speer RK73H1ETTP33R0F
- R118, R129, R137: symbol Auto_Library_WUT:KOA Speer RK73H1ETTP1002F -> Preferred_WUT:KOA Speer RK73H1ETTP1002F
- R89, R90: symbol Auto_Library_WUT:KOA Speer RK73H1ETTP1000F -> Preferred_WUT:KOA Speer RK73H1ETTP1000F
Changed lines of the file:
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@@
     )
   )
-  (symbol (lib_id "Auto_Library_WUT:KOA Speer RK73H1ETTP33R0F") (at 218.44 137.16 90) (unit 1)
+  (symbol (lib_id "Preferred_WUT:KOA Speer RK73H1ETTP33R0F") (at 218.44 137.16 90) (unit 1)
     (in_bom yes) (on_board yes) (dnp no) (fields_autoplaced)
     (property "Reference" "R110" (at 218.44 130.81 90)
@@
     )
   )
-  (symbol (lib_id "Auto_Library_WUT:Yageo CC0402KRX7R8BB104") (at 228.6 219.71 90) (unit 1)
+  (symbol (lib_id "Preferred_WUT:Yageo CC0402KRX7R8BB104") (at 228.6 219.71 90) (unit 1)
     (in_bom yes) (on_board yes) (dnp no)
     (property "Reference" "C35" (at 224.79 218.44 90) (do_not_autoplace)
@@
     )
     (property "Voltage" "25V" (at 231.14 217.17 0) (do_not_autoplace)
-      (effects (font (size 1.27 1.27) (color 0 100 100 1)) (justify left) hide)
+      (effects (font (size 1.27 1.27) (color 0 100 100 1)) (justify left))
     )
     (property "Manufacturer" "Yageo" (at 228.6 219.71 0)
@@
     )
   )
-  (symbol (lib_id "Auto_Library_WUT:Samsung Electro-Mechanics CL10A106MO8NQNC") (at 120.65 95.25 0) (unit 1)
+  (symbol (lib_id "Preferred_WUT:Samsung Electro-Mechanics CL10A106MO8NQNC") (at 120.65 95.25 0) (unit 1)
     (in_bom yes) (on_board yes) (dnp no) (fields_autoplaced)
     (property "Reference" "C15" (at 123.19 92.71 0) (do_not_autoplace)
@@
     )
   )
-  (symbol (lib_id "Auto_Library_WUT:KOA Speer RK73H1ETTP1002F") (at 176.53 241.3 180) (unit 1)
+  (symbol (lib_id "Preferred_WUT:KOA Speer RK73H1ETTP1002F") (at 176.53 241.3 180) (unit 1)
     (in_bom yes) (on_board yes) (dnp no) (fields_autoplaced)
     (property "Reference" "R129" (at 179.07 240.03 0)
@@
     )
   )
-  (symbol (lib_id "Auto_Library_WUT:Samsung Electro-Mechanics CL10A106MO8NQNC") (at 133.35 95.25 0) (unit 1)
+  (symbol (lib_id "Preferred_WUT:Samsung Electro-Mechanics CL10A106MO8NQNC") (at 133.35 95.25 0) (unit 1)
     (in_bom yes) (on_board yes) (dnp no) (fields_autoplaced)
     (property "Reference" "C17" (at 135.89 92.71 0) (do_not_autoplace)
@@
     )
   )
-  (symbol (lib_id "Auto_Library_WUT:Yageo CC0402KRX7R8BB104") (at 332.74 90.17 0) (unit 1)
+  (symbol (lib_id "Preferred_WUT:Yageo CC0402KRX7R8BB104") (at 332.74 90.17 0) (unit 1)
     (in_bom yes) (on_board yes) (dnp no) (fields_autoplaced)
     (property "Reference" "C9" (at 335.28 87.63 0) (do_not_autoplace)
@@
     )
   )
-  (symbol (lib_id "Auto_Library_WUT:Murata BLM18AG601SN1D") (at 43.18 88.9 0) (unit 1)
+  (symbol (lib_id "Preferred_WUT:Murata BLM18AG601SN1D") (at 43.18 88.9 0) (unit 1)
     (in_bom yes) (on_board yes) (dnp no) (fields_autoplaced)
     (property "Reference" "FB26" (at 43.1419 82.55 0)
@@
     )
   )
-  (symbol (lib_id "Auto_Library_WUT:Yageo CC0402KRX7R8BB104") (at 320.04 71.12 0) (unit 1)
+  (symbol (lib_id "Preferred_WUT:Yageo CC0402KRX7R8BB104") (at 320.04 71.12 0) (unit 1)
     (in_bom yes) (on_board yes) (dnp no) (fields_autoplaced)
     (property "Reference" "C9" (at 322.58 68.58 0) (do_not_autoplace)
@@
     )
   )
-  (symbol (lib_id "Auto_Library_WUT:Samsung Electro-Mechanics CL10A106MO8NQNC") (at 288.29 90.17 0) (unit 1)
+  (symbol (lib_id "Preferred_WUT:Samsung Electro-Mechanics CL10A106MO8NQNC") (at 288.29 90.17 0) (unit 1)
     (in_bom yes) (on_board yes) (dnp no) (fields_autoplaced)
     (property "Reference" "C7" (at 290.83 87.63 0) (do_not_autoplace)
@@
     )
   )
-  (symbol (lib_id "Auto_Library_WUT:Yageo CC0402KRX7R8BB104") (at 119.38 148.59 0) (unit 1)
+  (symbol (lib_id "Preferred_WUT:Yageo CC0402KRX7R8BB104") (at 119.38 148.59 0) (unit 1)
     (in_bom yes) (on_board yes) (dnp no) (fields_autoplaced)
     (property "Reference" "C159" (at 121.92 146.05 0) (do_not_autoplace)
@@
     )
   )
-  (symbol (lib_id "Auto_Library_WUT:Littelfuse AQ3522-01LTG") (at 294.64 219.71 90) (unit 1)
+  (symbol (lib_id "Preferred_WUT:Littelfuse AQ3522-01LTG") (at 294.64 219.71 90) (unit 1)
     (in_bom yes) (on_board yes) (dnp no) (fields_autoplaced)
     (property "Reference" "D9" (at 297.18 218.186 90)
@@
     )
   )
-  (symbol (lib_id "Auto_Library_WUT:KOA Speer RK73H1ETTP33R0F") (at 218.44 55.88 90) (unit 1)
+  (symbol (lib_id "Preferred_WUT:KOA Speer RK73H1ETTP33R0F") (at 218.44 55.88 90) (unit 1)
     (in_bom yes) (on_board yes) (dnp no) (fields_autoplaced)
     (property "Reference" "R100" (at 218.44 49.53 90)
@@
     )
   )
-  (symbol (lib_id "Auto_Library_WUT:Samsung Electro-Mechanics CL10A106MO8NQNC") (at 46.99 95.25 0) (unit 1)
+  (symbol (lib_id "Preferred_WUT:Samsung Electro-Mechanics CL10A106MO8NQNC") (at 46.99 95.25 0) (unit 1)
     (in_bom yes) (on_board yes) (dnp no) (fields_autoplaced)
     (property "Reference" "C7" (at 49.53 92.71 0) (do_not_autoplace)
@@
     )
   )
-  (symbol (lib_id "Auto_Library_WUT:KOA Speer RK73H1ETTP33R0F") (at 218.44 149.86 90) (unit 1)
+  (symbol (lib_id "Preferred_WUT:KOA Speer RK73H1ETTP33R0F") (at 218.44 149.86 90) (unit 1)
     (in_bom yes) (on_board yes) (dnp no) (fields_autoplaced)
     (property "Reference" "R111" (at 218.44 143.51 90)
@@
     )
   )
-  (symbol (lib_id "Auto_Library_WUT:KOA Speer RK73H1ETTP33R0F") (at 218.44 96.52 90) (unit 1)
+  (symbol (lib_id "Preferred_WUT:KOA Speer RK73H1ETTP33R0F") (at 218.44 96.52 90) (unit 1)
     (in_bom yes) (on_board yes) (dnp no) (fields_autoplaced)
     (property "Reference" "R105" (at 218.44 90.17 90)
@@
     )
   )
-  (symbol (lib_id "Auto_Library_WUT:KOA Speer RK73H1ETTP33R0F") (at 218.44 68.58 90) (unit 1)
+  (symbol (lib_id "Preferred_WUT:KOA Speer RK73H1ETTP33R0F") (at 218.44 68.58 90) (unit 1)
     (in_bom yes) (on_board yes) (dnp no) (fields_autoplaced)
     (property "Reference" "R101" (at 218.44 62.23 90)
@@
     )
   )
-  (symbol (lib_id "Auto_Library_WUT:Ekinglux_E6C0603VGAC1UDA") (at 176.53 250.19 270) (unit 1)
+  (symbol (lib_id "Preferred_WUT:Ekinglux_E6C0603VGAC1UDA") (at 176.53 250.19 270) (unit 1)
     (in_bom yes) (on_board yes) (dnp no) (fields_autoplaced)
     (property "Reference" "LD8" (at 180.34 248.6025 90)
@@
     )
   )
-  (symbol (lib_id "Auto_Library_WUT:Yageo CC0402KRX7R8BB104") (at 259.08 173.99 0) (unit 1)
+  (symbol (lib_id "Preferred_WUT:Yageo CC0402KRX7R8BB104") (at 259.08 173.99 0) (unit 1)
     (in_bom yes) (on_board yes) (dnp no) (fields_autoplaced)
     (property "Reference" "C9" (at 261.62 171.45 0) (do_not_autoplace)
@@
     )
   )
-  (symbol (lib_id "Auto_Library_WUT:KOA Speer RK73H1ETTP1000F") (at 129.54 123.19 90) (unit 1)
+  (symbol (lib_id "Preferred_WUT:KOA Speer RK73H1ETTP1000F") (at 129.54 123.19 90) (unit 1)
     (in_bom yes) (on_board yes) (dnp no) (fields_autoplaced)
     (property "Reference" "R90" (at 129.54 116.84 90)
@@
     )
   )
-  (symbol (lib_id "Auto_Library_WUT:KOA Speer RK73H1ETTP33R0F") (at 218.44 109.22 90) (unit 1)
+  (symbol (lib_id "Preferred_WUT:KOA Speer RK73H1ETTP33R0F") (at 218.44 109.22 90) (unit 1)
     (in_bom yes) (on_board yes) (dnp no) (fields_autoplaced)
     (property "Reference" "R106" (at 218.44 102.87 90)
@@
     )
   )
-  (symbol (lib_id "Auto_Library_WUT:KOA Speer RK73H1ETTP1002F") (at 247.65 173.99 0) (unit 1)
+  (symbol (lib_id "Preferred_WUT:KOA Speer RK73H1ETTP1002F") (at 247.65 173.99 0) (unit 1)
     (in_bom yes) (on_board yes) (dnp no) (fields_autoplaced)
     (property "Reference" "R118" (at 250.19 172.72 0)
@@
     )
   )
-  (symbol (lib_id "Auto_Library_WUT:Murata BLM18AG601SN1D") (at 284.48 83.82 0) (unit 1)
+  (symbol (lib_id "Preferred_WUT:Murata BLM18AG601SN1D") (at 284.48 83.82 0) (unit 1)
     (in_bom yes) (on_board yes) (dnp no) (fields_autoplaced)
     (property "Reference" "FB27" (at 284.4419 77.47 0)
@@
     )
   )
-  (symbol (lib_id "Auto_Library_WUT:KOA Speer RK73H1ETTP1000F") (at 208.28 219.71 0) (unit 1)
+  (symbol (lib_id "Preferred_WUT:KOA Speer RK73H1ETTP1000F") (at 208.28 219.71 0) (unit 1)
     (in_bom yes) (on_board yes) (dnp yes) (fields_autoplaced)
     (property "Reference" "R89" (at 210.82 218.44 0)
@@
     )
   )
-  (symbol (lib_id "Auto_Library_WUT:Yageo CC0402KRX7R8BB104") (at 58.42 101.6 0) (unit 1)
+  (symbol (lib_id "Preferred_WUT:Yageo CC0402KRX7R8BB104") (at 58.42 101.6 0) (unit 1)
     (in_bom yes) (on_board yes) (dnp no) (fields_autoplaced)
     (property "Reference" "C9" (at 60.96 99.06 0) (do_not_autoplace)
@@
     )
   )
-  (symbol (lib_id "Auto_Library_WUT:KOA Speer RK73H1ETTP1002F") (at 107.95 148.59 0) (unit 1)
+  (symbol (lib_id "Preferred_WUT:KOA Speer RK73H1ETTP1002F") (at 107.95 148.59 0) (unit 1)
     (in_bom yes) (on_board yes) (dnp no) (fields_autoplaced)
     (property "Reference" "R137" (at 110.49 147.32 0)
@@
     )
   )
-  (symbol (lib_id "Auto_Library_WUT:Samsung Electro-Mechanics CL10A106MO8NQNC") (at 320.04 90.17 0) (unit 1)
+  (symbol (lib_id "Preferred_WUT:Samsung Electro-Mechanics CL10A106MO8NQNC") (at 320.04 90.17 0) (unit 1)
     (in_bom yes) (on_board yes) (dnp no) (fields_autoplaced)
     (property "Reference" "C7" (at 322.58 87.63 0) (do_not_autoplace)
@@
     )
   )
-  (symbol (lib_id "Auto_Library_WUT:Yageo CC0402KRX7R8BB104") (at 139.7 217.17 0) (unit 1)
+  (symbol (lib_id "Preferred_WUT:Yageo CC0402KRX7R8BB104") (at 139.7 217.17 0) (unit 1)
     (in_bom yes) (on_board yes) (dnp no) (fields_autoplaced)
     (property "Reference" "C157" (at 142.24 214.63 0) (do_not_autoplace)
@@
     )
   )
-  (symbol (lib_id "Auto_Library_WUT:Yageo CC0402KRX7R8BB104") (at 300.99 90.17 0) (unit 1)
+  (symbol (lib_id "Preferred_WUT:Yageo CC0402KRX7R8BB104") (at 300.99 90.17 0) (unit 1)
     (in_bom yes) (on_board yes) (dnp no) (fields_autoplaced)
     (property "Reference" "C9" (at 303.53 87.63 0) (do_not_autoplace)

Commit message: Started placement
Parts:
- removed C17: 10u, Capacitor_SMD:C_0603_1608Metric, symbol Preferred_WUT:Samsung Electro-Mechanics CL10A106MO8NQNC
- added C24: 100n, Capacitor_SMD:C_0402_1005Metric, symbol Preferred_WUT:Yageo CC0402KRX7R8BB104
Connections:
- net 0V: now also C24.2
- net at C13.1, C15.1, R20.1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: now also C24.1
Changed lines of the file:
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@@
-    )
-  )
-  (symbol (lib_id "Preferred_WUT:Samsung Electro-Mechanics CL10A106MO8NQNC") (at 133.35 95.25 0) (unit 1)
-    (in_bom yes) (on_board yes) (dnp no) (fields_autoplaced)
-    (property "Reference" "C17" (at 135.89 92.71 0) (do_not_autoplace)
-      (effects (font (size 1.27 1.27)) (justify left))
-    )
-    (property "Value" "10u" (at 135.89 95.25 0) (do_not_autoplace)
-      (effects (font (size 1.27 1.27)) (justify left))
-    )
-    (property "Footprint" "Capacitor_SMD:C_0603_1608Metric" (at 133.35 95.25 0)
-      (effects (font (size 1.27 1.27)) hide)
-    )
-    (property "Datasheet" "https://www.mouser.co.uk/datasheet/2/585/MLCC-1837944.pdf" (at 133.35 95.25 0)
-      (effects (font (size 1.27 1.27)) hide)
-    )
-    (property "Voltage" "16V" (at 135.89 97.79 0) (do_not_autoplace)
-      (effects (font (size 1.27 1.27) (color 0 100 100 1)) (justify left))
-    )
-    (property "Manufacturer" "Samsung Electro-Mechanics" (at 133.35 95.25 0)
-      (effects (font (size 1.27 1.27)) hide)
-    )
-    (property "MPN" "CL10A106MO8NQNC" (at 133.35 95.25 0)
-      (effects (font (size 1.27 1.27)) hide)
-    )
-    (property "Tolerance" "20%" (at 133.35 95.25 0)
-      (effects (font (size 1.27 1.27)) hide)
-    )
-    (property "Dielectric" "X5R" (at 133.35 95.25 0)
-      (effects (font (size 1.27 1.27)) hide)
-    )
-    (property "Height" "0.9mm" (at 133.35 95.25 0)
-      (effects (font (size 1.27 1.27)) hide)
-    )
-    (pin "1")
-    (pin "2")
-    (instances
-      (project "Master Timing Card"
-        (path "/6e8e281e-e30f-459d-852f-231836068db5/231ba923-6354-4319-a55b-e8f523b1b9f4"
-          (reference "C17") (unit 1)
-        )
-        (path "/6e8e281e-e30f-459d-852f-231836068db5/4066cd97-f2f5-4d90-9329-88af4fe2410f"
-          (reference "C33") (unit 1)
-        )
-      )
     )
   )
@@
         )
       )
+    )
+  )
+  (symbol (lib_id "Preferred_WUT:Yageo CC0402KRX7R8BB104") (at 133.35 95.25 0) (unit 1)
+    (in_bom yes) (on_board yes) (dnp no) (fields_autoplaced)
+    (property "Reference" "C24" (at 135.89 92.71 0) (do_not_autoplace)
+      (effects (font (size 1.27 1.27)) (justify left))
+    )
+    (property "Value" "100n" (at 135.89 95.25 0) (do_not_autoplace)
+      (effects (font (size 1.27 1.27)) (justify left))
+    )
+    (property "Footprint" "Capacitor_SMD:C_0402_1005Metric" (at 133.35 95.25 0)
+      (effects (font (size 1.27 1.27)) hide)
+    )
+    (property "Datasheet" "https://www.yageo.com/upload/media/product/productsearch/datasheet/mlcc/UPY-GPHC_X7R_6.3V-to-250V_23.pdf" (at 133.35 95.25 0)
+      (effects (font (size 1.27 1.27)) hide)
+    )
+    (property "Voltage" "25V" (at 135.89 97.79 0) (do_not_autoplace)
+      (effects (font (size 1.27 1.27) (color 0 100 100 1)) (justify left))
+    )
+    (property "Manufacturer" "Yageo" (at 133.35 95.25 0)
+      (effects (font (size 1.27 1.27)) hide)
+    )
+    (property "MPN" "CC0402KRX7R8BB104" (at 133.35 95.25 0)
+      (effects (font (size 1.27 1.27)) hide)
+    )
+    (property "Tolerance" "10%" (at 133.35 95.25 0)
+      (effects (font (size 1.27 1.27)) hide)
+    )
+    (property "Dielectric" "X7R" (at 133.35 95.25 0)
+      (effects (font (size 1.27 1.27)) hide)
+    )
+    (property "Height" "0.5mm" (at 133.35 95.25 0)
+      (effects (font (size 1.27 1.27)) hide)
+    )
+    (pin "1")
+    (pin "2")
+    (instances
+      (project "Master Timing Card"
+        (path "/6e8e281e-e30f-459d-852f-231836068db5/4066cd97-f2f5-4d90-9329-88af4fe2410f"
+          (reference "C24") (unit 1)
+        )
+      )
