File: pll.kicad_sch (KiCad schematic)
At the start: 63 parts, among them CN11 UE75-A20-6000T, CN12 U77-A1114-30L1, CN15 731385033, Q6 DMN62D0U-7, T4 TC2-72T+, U11 SY75576LKY, U15 SN74LVC1G02DCK, U3 TI TPS79301DBV

Commit message: initial placement
Parts:
- added R25, R26: 10k, Resistor_SMD:R_0402_1005Metric, symbol Preferred_WUT:KOA Speer RK73H1ETTP1002F
Connections:
- net 3V3: now also R25.1, R26.1
- net Frequency Synthesiser 1/~{PLL_LOCK_OD}: now also R25.2
- net Frequency Synthesiser 2/~{PLL_LOCK_OD}: now also R26.2
Other:
- moved on the sheet: C157, U15

Commit message: layout progress
Parts:
- removed R89: 100R, Resistor_SMD:R_0402_1005Metric, symbol Preferred_WUT:KOA Speer RK73H1ETTP1000F
- C11, C22, C27: renamed from C7; symbol Preferred_WUT:Samsung Electro-Mechanics CL10A106MO8NQNC -> AAA_Preferred_WUT:Samsung Electro-Mechanics CL10A106MO8NQNC
- C12, C21, C23, C26, C29: renamed from C9; symbol Preferred_WUT:Yageo CC0402KRX7R8BB104 -> AAA_Preferred_WUT:Yageo CC0402KRX7R8BB104
- C13: renamed from C154; symbol Preferred_WUT:Yageo CC0402KRX7R8BB104 -> AAA_Preferred_WUT:Yageo CC0402KRX7R8BB104
- C15: symbol Preferred_WUT:Samsung Electro-Mechanics CL10A106MO8NQNC -> AAA_Preferred_WUT:Samsung Electro-Mechanics CL10A106MO8NQNC
- C16: renamed from C159; symbol Preferred_WUT:Yageo CC0402KRX7R8BB104 -> AAA_Preferred_WUT:Yageo CC0402KRX7R8BB104
- C17: renamed from C24; symbol Preferred_WUT:Yageo CC0402KRX7R8BB104 -> AAA_Preferred_WUT:Yageo CC0402KRX7R8BB104
- C18: renamed from C33; symbol Preferred_WUT:Yageo CC0402KRX7R8BB104 -> AAA_Preferred_WUT:Yageo CC0402KRX7R8BB104
- C19: renamed from C157; symbol Preferred_WUT:Yageo CC0402KRX7R8BB104 -> AAA_Preferred_WUT:Yageo CC0402KRX7R8BB104
- C20: renamed from C35; symbol Preferred_WUT:Yageo CC0402KRX7R8BB104 -> AAA_Preferred_WUT:Yageo CC0402KRX7R8BB104
- D18: renamed from D9; symbol Preferred_WUT:Littelfuse AQ3522-01LTG -> AAA_Preferred_WUT:Littelfuse AQ3522-01LTG
- FB2: renamed from FB26; symbol Preferred_WUT:Murata BLM18AG601SN1D -> AAA_Preferred_WUT:Murata BLM18AG601SN1D
- FB3: renamed from FB27; symbol Preferred_WUT:Murata BLM18AG601SN1D -> AAA_Preferred_WUT:Murata BLM18AG601SN1D
- LD5: renamed from LD8; symbol Preferred_WUT:Ekinglux_E6C0603VGAC1UDA -> AAA_Preferred_WUT:Ekinglux_E6C0603VGAC1UDA
- Q1: renamed from Q6; symbol FET_WUT:DMN62D0U-7 -> Transistor_WUT:Diodes-Inc_DMN62D0U-7
- R43: renamed from R137; symbol Preferred_WUT:KOA Speer RK73H1ETTP1002F -> AAA_Preferred_WUT:KOA Speer RK73H1ETTP1002F
- R44: renamed from R90; symbol Preferred_WUT:KOA Speer RK73H1ETTP1000F -> AAA_Preferred_WUT:KOA Speer RK73H1ETTP1000F
- R45: renamed from R25; symbol Preferred_WUT:KOA Speer RK73H1ETTP1002F -> AAA_Preferred_WUT:KOA Speer RK73H1ETTP1002F
- R47: renamed from R26; symbol Preferred_WUT:KOA Speer RK73H1ETTP1002F -> AAA_Preferred_WUT:KOA Speer RK73H1ETTP1002F
- R48: renamed from R129; symbol Preferred_WUT:KOA Speer RK73H1ETTP1002F -> AAA_Preferred_WUT:KOA Speer RK73H1ETTP1002F
- R49: renamed from R100; symbol Preferred_WUT:KOA Speer RK73H1ETTP33R0F -> AAA_Preferred_WUT:KOA Speer RK73H1ETTP33R0F
- R50: renamed from R101; symbol Preferred_WUT:KOA Speer RK73H1ETTP33R0F -> AAA_Preferred_WUT:KOA Speer RK73H1ETTP33R0F
- R51: renamed from R105; symbol Preferred_WUT:KOA Speer RK73H1ETTP33R0F -> AAA_Preferred_WUT:KOA Speer RK73H1ETTP33R0F
- R52: renamed from R106; symbol Preferred_WUT:KOA Speer RK73H1ETTP33R0F -> AAA_Preferred_WUT:KOA Speer RK73H1ETTP33R0F
- R53: renamed from R110; symbol Preferred_WUT:KOA Speer RK73H1ETTP33R0F -> AAA_Preferred_WUT:KOA Speer RK73H1ETTP33R0F
- R54: renamed from R111; symbol Preferred_WUT:KOA Speer RK73H1ETTP33R0F -> AAA_Preferred_WUT:KOA Speer RK73H1ETTP33R0F
- R58: renamed from R118; symbol Preferred_WUT:KOA Speer RK73H1ETTP1002F -> AAA_Preferred_WUT:KOA Speer RK73H1ETTP1002F
- renumbered C13 to C14, C112 to C24, C110 to C25, C109 to C28, CN12 to CN10, CN15 to CN9, H1 to H2, L6 to L1, L5 to L2, R107 to R37, R91 to R38, R108 to R39, R92 to R40, R20 to R41, R21 to R42, R94 to R46, R102 to R55, R104 to R56, R103 to R57, R97 to R59, R99 to R60, R98 to R61, R95 to R62, R96 to R63, T4 to T1, TP4 to TP2, U3 to U4, U11 to U5, U15 to U6
Connections:
- net 0V: now also T1.4; no longer T1.6
- net CLKD_N: now also T1.3; no longer T1.1
- net CLKD_P: now also T1.1; no longer T1.3
- net at R59.1: now also T1.6; no longer T1.4
Other:
- note removed: "Either fit this resistor or components for additonal 10MHz out"
- moved on the sheet: C21, R58, T1

Commit message: less than 100 tracks to go!
Parts:
- added C164: 100n, Capacitor_SMD:C_0402_1005Metric, symbol AAA_Preferred_WUT:Yageo CC0402KRX7R8BB104
- added R125, R126: 33R, Resistor_SMD:R_0402_1005Metric, symbol AAA_Preferred_WUT:KOA Speer RK73H1ETTP33R0F
Connections:
- net 0V: now also T1.2; no longer C20.1
- net CLKB_N: now also R126.1; no longer R52.1
- net CLKB_P: now also R125.1; no longer R51.1
- net CLKC_N: now also R52.1; no longer R54.1
- net CLKC_P: now also R51.1; no longer R53.1
- net CLKD_N: now also R54.1; no longer T1.3
- net CLKD_P: now also R53.1; no longer T1.1
- net Frequency Synthesiser 1/~{PLL_LOCK_OD}: now also U6.2; no longer U6.1
- net Frequency Synthesiser 2/~{PLL_LOCK_OD}: now also U6.1; no longer U6.2
- net at C20.2: now also T1.1; no longer T1.2
- new net: C164.2, T1.3
- new net EXT_CLK_N: C164.1, R126.2
- new net EXT_CLK_P: C20.1, R125.2
Other:
- moved on the sheet: R49, R50, R51, R52, R53, R54, R55, R56, R57

Commit message: committing before attempting scripting
Parts:
- renumbered C164 to C21, C21 to C22, C22 to C23, C23 to C24, C24 to C25, C25 to C26, C26 to C27, C27 to C28, C28 to C29, C29 to C30, R55 to R51, R56 to R52, R57 to R53, R125 to R54, R126 to R55, R51 to R56, R52 to R57, R53 to R58, R54 to R59, R58 to R60, R59 to R61, R60 to R62, R61 to R63, R62 to R64, R63 to R65
