File: Master Timing Card.kicad_pcb (KiCad board)
At the start: 4 copper layers, 170 x 100 mm, 418 parts, among them CN10 M2 x 2.5mm, CN11 UE75-A20-6000T, CN12 U77-A1114-30L1, CN13 Harwin M20-9990246, CN14 USB4110-GF-A, CN15 731385033, CN2 Samtec GRF1-J-P-08-E-RA-TH1, CN3 Amphenol 86093488613755E1LF, CN7 104031-0811, CN9 TE 1-2199230-6, J1 Connector_RJ45_Magjack_Abraco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, Q1 DMN62D0U-7, Q2 DMN62D0U-7, Q3 DMN62D0U-7, Q4 onsemi FDC6330L, Q5 TSM085P03CV RGG, Q6 DMN62D0U-7, T1 TC2-72T+, T2 TC2-72T+, T3 TC2-72T+, T4 TC2-72T+, T5 TC2-72T+, T6 TC2-72T+, T7 TC2-72T+, T8 TC2-72T+, T9 TC2-72T+, U1 DS2431P+, U10 INA3221AIRGV, U11 SY75576LKY, U12 TI TPS79301DBV, U13 LT3045IDD#PBF, U14 LT3045IDD#PBF, U15 SN74LVC1G02DCK, U16 SN74LVC2G157DCU, U17 ZED-F9T-10B, U2 Analog MAX3483ESA+, U3 TI TPS79301DBV, U4 TI TPS79301DBV, U5 RC32504A000GNK#BB0, U6 RC32504A000GNK#BB0, U7 SN74LVC1G125DBV, U8 SN74LVC1G125DBV, U9 Analog LT8650SEV#PBF

Commit message: Moved to discrete GPS
Parts:
- removed C14: 15p, Capacitor_SMD:C_0402_1005Metric
- removed C23: 100n, Capacitor_SMD:C_0402_1005Metric
- removed C4: 4n7, Capacitor_SMD:C_0402_1005Metric
- removed F2: 250mA, Fuse:Fuse_0603_1608Metric
- removed FB7: 1k8, Inductor_SMD:L_0402_1005Metric
- removed Q1: DMN62D0U-7, Package_TO_SOT_SMD:SOT-23
- removed R25, R27: 10k, Resistor_SMD:R_0402_1005Metric
- removed R26: 100R, Resistor_SMD:R_0402_1005Metric
- removed TP2: ~, TestPoint:TestPoint_Pad_D1.0mm
- added C156: 100n, Capacitor_SMD:C_0402_1005Metric, F.Cu at (51.5, 108.8)
- added C168: 4n7, Capacitor_SMD:C_0402_1005Metric, F.Cu at (51.5, 107.8)
- added C169: 10u, Capacitor_SMD:C_0603_1608Metric, F.Cu at (50.0, 113.2)
- added CN1: CONSMA002-L-G, Connector_WUT:SMA_Linx_CONSMA002-L-G_Horizontal, F.Cu at (44.6, 106.5)
- added D20: 5V0, Diode_SMD:D_SOD-523, F.Cu at (50.5, 105.0)
- added L1: 47n, Inductor_SMD:L_0402_1005Metric, F.Cu at (52.0, 106.2)
- added Q10: MMBT2907A-7-F, Package_TO_SOT_SMD:SOT-23, F.Cu at (53.2, 111.5)
- added Q7: DMN62D0U-7, Package_TO_SOT_SMD:SOT-23, F.Cu at (76.2, 103.8)
- added Q9: MMBT2907A-7-F, Package_TO_SOT_SMD:SOT-23, F.Cu at (53.2, 117.5)
- added R109: 100R, Resistor_SMD:R_0402_1005Metric, F.Cu at (50.2, 110.5)
- added R112: 10k, Resistor_SMD:R_0402_1005Metric, F.Cu at (42.2, 113.5)
- added R113: 1k0, Resistor_SMD:R_0402_1005Metric, F.Cu at (53.2, 120.5)
- added R114: 10R, Resistor_SMD:R_0805_2012Metric, F.Cu at (53.2, 114.5)
- added R123: 10k, Resistor_SMD:R_0402_1005Metric, F.Cu at (41.7, 112.0)
- added R124: 22k, Resistor_SMD:R_0402_1005Metric, F.Cu at (42.7, 112.0)
- added R125: 10k, Resistor_SMD:R_0402_1005Metric, F.Cu at (79.7, 103.8)
- added TP5: ~, TestPoint:TestPoint_Pad_D1.0mm, B.Cu at (62.5, 102.5)
- added U18: TLV7031DCK, Package_TO_SOT_SMD:SOT-353_SC-70-5, F.Cu at (44.7, 112.5)
- C19, C39: value 4n7 -> 100n
- C20: value 10u -> 100n; footprint Capacitor_SMD:C_0603_1608Metric -> Capacitor_SMD:C_0402_1005Metric
- FB6: value 600R -> 1k8; footprint Inductor_SMD:L_0603_1608Metric -> Inductor_SMD:L_0402_1005Metric
- R22: value 20k -> 22k
- R23: value 6k8 -> 7k5
- moved D1 168.6 mm to (268.2, 112.6), turned to 90 degrees
- moved C116 166.5 mm to (268.2, 115.3), turned to -90 degrees
- moved R49 165.6 mm to (263.7, 109.8), turned to 180 degrees
- moved Q4 163.3 mm to (263.7, 112.6), turned to 90 degrees
- moved C117 160.6 mm to (263.2, 115.3), turned to 180 degrees
- moved R50 160.5 mm to (261.2, 112.6), turned to -90 degrees
- moved CN7 159.8 mm to (268.2, 124.8), turned to 180 degrees
- moved D2 159.4 mm to (263.2, 116.8), turned to 180 degrees
- moved C55 86.9 mm to (252.5, 66.0)
- moved C56 86.9 mm to (252.5, 68.0)
- moved C57 86.9 mm to (252.5, 69.9)
- moved C58 86.9 mm to (252.5, 71.9)
- moved C59 86.9 mm to (252.5, 73.9)
- moved C60 86.9 mm to (252.5, 75.8)
- moved C61 86.9 mm to (252.5, 77.8)
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Connections:
- C13 pad 1: Net-(U3-OUT) -> Net-(U17-V_BCKP)
- C15 pad 1: Net-(U3-OUT) -> Net-(U17-V_BCKP)
- C17 pad 1: Net-(U3-OUT) -> Net-(U17-V_BCKP)
- C18 pad 1: Net-(C18-Pad1) -> 3V3
- C19 pad 1: /GPS/VCC_ANT -> /GPS/GNSS_RESET
- C20 pad 1: /GPS/VCC_GNSS -> Net-(U17-V_BCKP)
- C21 pad 1: /GPS/VCC_GNSS -> Net-(U17-V_BCKP)
- C39 pad 1: /GPS/VCC_GNSS -> Net-(U17-V_BCKP)
- C5 pad 1: /GPS/GNSS_TX_M -> Net-(U17-TXD/SPI_MISO)
- C6 pad 1: /GPS/GNSS_RX_M -> Net-(U17-RXD/SPI_MOSI)
- FB2 pad 2: /GPS/GNSS_TX_M -> Net-(U17-TXD/SPI_MISO)
- FB3 pad 2: /GPS/GNSS_RX_M -> Net-(U17-RXD/SPI_MOSI)
- FB6 pad 1: Net-(U3-OUT) -> Net-(Q9-E)
- FB6 pad 2: /GPS/VCC_GNSS -> Net-(U4-OUT)
- R20 pad 1: Net-(U3-OUT) -> Net-(U17-V_BCKP)
- R88 pad 1: Net-(C18-Pad1) -> Net-(U4-OUT)
- TP1 pad 1: Net-(U3-OUT) -> Net-(U17-V_BCKP)
- U17 pad 2: unconnected-(U17-RF_IN-Pad2) -> Net-(CN1-In)
- U17 pad 33: unconnected-(U17-VCC-Pad33) -> Net-(U17-V_BCKP)
- U17 pad 34: unconnected-(U17-VCC-Pad34) -> Net-(U17-V_BCKP)
- U17 pad 36: unconnected-(U17-V_BCKP-Pad36) -> Net-(U17-V_BCKP)
- U17 pad 38: unconnected-(U17-V_USB-Pad38) -> 0V
- U17 pad 42: unconnected-(U17-TXD/SPI_MISO-Pad42) -> Net-(U17-TXD/SPI_MISO)
- U17 pad 43: unconnected-(U17-RXD/SPI_MOSI-Pad43) -> Net-(U17-RXD/SPI_MOSI)
- U17 pad 49: unconnected-(U17-~{RESET}-Pad49) -> Net-(Q7-D)
- U17 pad 50: unconnected-(U17-~{SAFEBOOT}-Pad50) -> Net-(U17-~{SAFEBOOT})
- U17 pad 53: unconnected-(U17-TIMEPULSE-Pad53) -> /GPS/GNSS_CLK_M
- U17 pad 54: unconnected-(U17-TIMEPULSE2-Pad54) -> /GPS/GNSS_PPS_M
- U17 pad 6: unconnected-(U17-ANT_SHORT_N-Pad6) -> /GPS/~{ANT_SHORT}
- U3 pad 6: Net-(U3-OUT) -> Net-(U17-V_BCKP)
Routing:
- net 0V: track 201.6 -> 179.1 mm, vias 196 -> 214
- net /CM4 Interfaces/SD_PWR_ON: track 25.2 -> 5.18 mm
- net Net-(CN1-In): track 0.00 -> 13.5 mm
- net /CM4 Interfaces/SD_CLK: track 12.1 -> 0.00 mm
- net Net-(U3-OUT): track 10.2 -> 0.00 mm
- net /CM4 Interfaces/SD_CMD: track 9.97 -> 0.00 mm
- net /CM4 Interfaces/SD_DAT0: track 11.4 -> 1.57 mm, vias 2 -> 1
- net /GPS/VCC_GNSS: track 8.58 -> 0.00 mm
- net /CM4 Interfaces/SD_DAT1: track 9.82 -> 1.70 mm
- net /CM4 Interfaces/SD_DAT3: track 8.01 -> 0.00 mm
- net Net-(LD9-Pad4): track 0.00 -> 7.64 mm
- net Net-(LD9-Pad1): track 0.00 -> 7.63 mm
- net Net-(Q10-C): track 0.00 -> 7.48 mm
- net Net-(LD9-Pad6): track 0.00 -> 6.39 mm
- net Net-(Q9-E): track 0.00 -> 5.77 mm
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
Commit message: initial placement
Parts:
- removed C102, C65: 4n7, Capacitor_SMD:C_0402_1005Metric
- removed C103, C66: 100n, Capacitor_SMD:C_0402_1005Metric
- removed Q2, Q3: DMN62D0U-7, Package_TO_SOT_SMD:SOT-23
- removed R28, R47: 10k, Resistor_SMD:R_0402_1005Metric
- removed R30, R48: 100R, Resistor_SMD:R_0402_1005Metric
- added R25: 10k, Resistor_SMD:R_0402_1005Metric, F.Cu at (107.8, 76.8)
- added R26: 10k, Resistor_SMD:R_0402_1005Metric, F.Cu at (107.8, 78.2)
- moved TP4 204.5 mm to (71.2, 78.8)
- moved R56 188.2 mm to (90.8, 72.2), turned to -90 degrees
- moved R35 184.3 mm to (91.8, 72.2), turned to 90 degrees
- moved R136 183.1 mm to (96.8, 74.2), turned to -90 degrees
- moved C70 182.8 mm to (61.0, 51.8)
- moved R34 181.9 mm to (92.8, 72.2), turned to 90 degrees
- moved R2 180.6 mm to (95.0, 42.3)
- moved R3 180.6 mm to (95.0, 44.2)
- moved R36 180.6 mm to (100.8, 44.2)
- moved R37 180.6 mm to (100.8, 46.2)
- moved R4 180.6 mm to (95.0, 46.2)
- moved R5 180.6 mm to (95.0, 48.2)
- moved R54 180.6 mm to (100.8, 52.2)
- moved R6 180.6 mm to (95.0, 50.2)
- moved R7 180.6 mm to (95.0, 52.2)
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Connections:
- R29 pad 2: Net-(Q2-G) -> /PLL and SFP/Frequency Synthesiser 1/~{PLL_LOCK_OD}
- R46 pad 2: Net-(Q3-G) -> /PLL and SFP/Frequency Synthesiser 2/~{PLL_LOCK_OD}
Routing:
- net 0V: track 179.1 -> 290.0 mm, vias 214 -> 319
- net /RF6: track 15.0 -> 45.0 mm, vias 1 -> 3
- net /RF7: track 15.0 -> 44.6 mm, vias 1 -> 3
- net /RF5: track 14.2 -> 42.5 mm, vias 1 -> 3
- net /RF8: track 17.7 -> 33.3 mm, vias 1 -> 3
- net /RF3: track 14.6 -> 29.6 mm, vias 1 -> 2
- net /RF2: track 15.0 -> 30.0 mm, vias 1 -> 2
- net /PLL and SFP/Frequency Synthesiser 2/RF1_N: track 0.00 -> 14.4 mm
- net /PLL and SFP/Frequency Synthesiser 2/RF4_N: track 0.00 -> 14.2 mm
- net /RF1: track 14.2 -> 28.3 mm, vias 1 -> 2
- net /PLL and SFP/Frequency Synthesiser 2/RF1_P: track 0.00 -> 13.7 mm
- net /PLL and SFP/Frequency Synthesiser 2/RF4_P: track 0.00 -> 13.5 mm
- net /PLL and SFP/Frequency Synthesiser 2/1V8_PLL: track 0.00 -> 11.9 mm, vias 0 -> 6
- net /PLL and SFP/Frequency Synthesiser 1/1V8_PLL: track 0.00 -> 11.9 mm, vias 0 -> 6
- net /RF4: track 15.0 -> 26.0 mm, vias 1 -> 2
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