File: cm4_gpio.kicad_sch (KiCad schematic)
At the start: 39 parts, among them CN13 Harwin M20-9990246, U8 SN74LVC1G125DBV

Commit message: Moved to preferred library
Parts:
- C116, C125: symbol Auto_Library_WUT:Yageo CC0402KRX7R8BB104 -> Preferred_WUT:Yageo CC0402KRX7R8BB104
- D7: symbol Auto_Library_WUT:nexperia PESD3V3U1UB,115 -> Preferred_WUT:nexperia PESD3V3U1UB,115
- LD1: symbol Auto_Library_WUT:Lite-On_LTST-C193KRKT-5A -> Preferred_WUT:Lite-On_LTST-C193KRKT-5A
- LD3: symbol Auto_Library_WUT:Ekinglux_E6C0603VGAC1UDA -> Preferred_WUT:Ekinglux_E6C0603VGAC1UDA
- R136, R14, R24, R33, R34, R36, R37, R5, R6, R60, R8, R9: symbol Auto_Library_WUT:KOA Speer RK73H1ETTP1000F -> Preferred_WUT:KOA Speer RK73H1ETTP1000F
- R52, R53, R56: symbol Auto_Library_WUT:KOA Speer RK73Z1ETTP -> Preferred_WUT:KOA Speer RK73Z1ETTP
- R54, R55: symbol Auto_Library_WUT:KOA Speer RK73H1ETTP1001F -> Preferred_WUT:KOA Speer RK73H1ETTP1001F
- R7: symbol Auto_Library_WUT:KOA Speer RK73H1ETTP33R0F -> Preferred_WUT:KOA Speer RK73H1ETTP33R0F
Changed lines of the file:
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@@
     )
   )
-  (symbol (lib_id "Auto_Library_WUT:KOA Speer RK73H1ETTP1000F") (at 231.14 58.42 90) (unit 1)
+  (symbol (lib_id "Preferred_WUT:KOA Speer RK73H1ETTP1000F") (at 231.14 58.42 90) (unit 1)
     (in_bom yes) (on_board yes) (dnp no)
     (property "Reference" "R5" (at 224.79 57.15 90)
@@
     )
   )
-  (symbol (lib_id "Auto_Library_WUT:KOA Speer RK73H1ETTP1000F") (at 175.26 76.2 90) (unit 1)
+  (symbol (lib_id "Preferred_WUT:KOA Speer RK73H1ETTP1000F") (at 175.26 76.2 90) (unit 1)
     (in_bom yes) (on_board yes) (dnp no)
     (property "Reference" "R6" (at 168.91 74.93 90)
@@
     )
   )
-  (symbol (lib_id "Auto_Library_WUT:Ekinglux_E6C0603VGAC1UDA") (at 265.43 139.7 270) (unit 1)
+  (symbol (lib_id "Preferred_WUT:Ekinglux_E6C0603VGAC1UDA") (at 265.43 139.7 270) (unit 1)
     (in_bom yes) (on_board yes) (dnp no)
     (property "Reference" "LD3" (at 267.97 139.7 90)
@@
     )
   )
-  (symbol (lib_id "Auto_Library_WUT:KOA Speer RK73H1ETTP1000F") (at 231.14 60.96 90) (unit 1)
+  (symbol (lib_id "Preferred_WUT:KOA Speer RK73H1ETTP1000F") (at 231.14 60.96 90) (unit 1)
     (in_bom yes) (on_board yes) (dnp no)
     (property "Reference" "R37" (at 224.79 59.69 90)
@@
     )
   )
-  (symbol (lib_id "Auto_Library_WUT:Yageo CC0402KRX7R8BB104") (at 127 118.11 0) (unit 1)
+  (symbol (lib_id "Preferred_WUT:Yageo CC0402KRX7R8BB104") (at 127 118.11 0) (unit 1)
     (in_bom yes) (on_board yes) (dnp no) (fields_autoplaced)
     (property "Reference" "C116" (at 129.54 115.57 0) (do_not_autoplace)
@@
     )
   )
-  (symbol (lib_id "Auto_Library_WUT:KOA Speer RK73H1ETTP33R0F") (at 175.26 86.36 270) (mirror x) (unit 1)
+  (symbol (lib_id "Preferred_WUT:KOA Speer RK73H1ETTP33R0F") (at 175.26 86.36 270) (mirror x) (unit 1)
     (in_bom yes) (on_board yes) (dnp no)
     (property "Reference" "R7" (at 168.91 85.09 90)
@@
     )
   )
-  (symbol (lib_id "Auto_Library_WUT:KOA Speer RK73H1ETTP1000F") (at 231.14 81.28 90) (unit 1)
+  (symbol (lib_id "Preferred_WUT:KOA Speer RK73H1ETTP1000F") (at 231.14 81.28 90) (unit 1)
     (in_bom yes) (on_board yes) (dnp no)
     (property "Reference" "R14" (at 224.79 80.01 90)
@@
     )
   )
-  (symbol (lib_id "Auto_Library_WUT:Yageo CC0402KRX7R8BB104") (at 177.8 160.02 0) (unit 1)
+  (symbol (lib_id "Preferred_WUT:Yageo CC0402KRX7R8BB104") (at 177.8 160.02 0) (unit 1)
     (in_bom yes) (on_board yes) (dnp no) (fields_autoplaced)
     (property "Reference" "C125" (at 180.34 157.48 0) (do_not_autoplace)
@@
     )
   )
-  (symbol (lib_id "Auto_Library_WUT:KOA Speer RK73H1ETTP1000F") (at 231.14 73.66 90) (unit 1)
+  (symbol (lib_id "Preferred_WUT:KOA Speer RK73H1ETTP1000F") (at 231.14 73.66 90) (unit 1)
     (in_bom yes) (on_board yes) (dnp no)
     (property "Reference" "R8" (at 224.79 72.39 90)
@@
     )
   )
-  (symbol (lib_id "Auto_Library_WUT:nexperia PESD3V3U1UB,115") (at 167.64 160.02 90) (unit 1)
+  (symbol (lib_id "Preferred_WUT:nexperia PESD3V3U1UB,115") (at 167.64 160.02 90) (unit 1)
     (in_bom yes) (on_board yes) (dnp no) (fields_autoplaced)
     (property "Reference" "D7" (at 170.18 158.496 90)
@@
     )
   )
-  (symbol (lib_id "Auto_Library_WUT:KOA Speer RK73Z1ETTP") (at 175.26 120.65 90) (unit 1)
+  (symbol (lib_id "Preferred_WUT:KOA Speer RK73Z1ETTP") (at 175.26 120.65 90) (unit 1)
     (in_bom yes) (on_board yes) (dnp no)
     (property "Reference" "R53" (at 171.45 119.38 90)
@@
     )
   )
-  (symbol (lib_id "Auto_Library_WUT:KOA Speer RK73H1ETTP1000F") (at 175.26 78.74 90) (unit 1)
+  (symbol (lib_id "Preferred_WUT:KOA Speer RK73H1ETTP1000F") (at 175.26 78.74 90) (unit 1)
     (in_bom yes) (on_board yes) (dnp no)
     (property "Reference" "R9" (at 168.91 77.47 90)
@@
     )
   )
-  (symbol (lib_id "Auto_Library_WUT:KOA Speer RK73H1ETTP1000F") (at 177.8 147.32 0) (unit 1)
+  (symbol (lib_id "Preferred_WUT:KOA Speer RK73H1ETTP1000F") (at 177.8 147.32 0) (unit 1)
     (in_bom yes) (on_board yes) (dnp no) (fields_autoplaced)
     (property "Reference" "R60" (at 180.34 146.05 0)
@@
     )
   )
-  (symbol (lib_id "Auto_Library_WUT:KOA Speer RK73Z1ETTP") (at 233.68 133.35 90) (unit 1)
+  (symbol (lib_id "Preferred_WUT:KOA Speer RK73Z1ETTP") (at 233.68 133.35 90) (unit 1)
     (in_bom yes) (on_board yes) (dnp no)
     (property "Reference" "R56" (at 229.87 132.08 90)
@@
     )
   )
-  (symbol (lib_id "Auto_Library_WUT:KOA Speer RK73H1ETTP1001F") (at 114.3 133.35 90) (unit 1)
+  (symbol (lib_id "Preferred_WUT:KOA Speer RK73H1ETTP1001F") (at 114.3 133.35 90) (unit 1)
     (in_bom yes) (on_board yes) (dnp no) (fields_autoplaced)
     (property "Reference" "R55" (at 114.3 127 90)
@@
     )
   )
-  (symbol (lib_id "Auto_Library_WUT:KOA Speer RK73H1ETTP1000F") (at 231.14 66.04 90) (unit 1)
+  (symbol (lib_id "Preferred_WUT:KOA Speer RK73H1ETTP1000F") (at 231.14 66.04 90) (unit 1)
     (in_bom yes) (on_board yes) (dnp no)
     (property "Reference" "R36" (at 224.79 64.77 90)
@@
     )
   )
-  (symbol (lib_id "Auto_Library_WUT:KOA Speer RK73H1ETTP1000F") (at 231.14 83.82 90) (unit 1)
+  (symbol (lib_id "Preferred_WUT:KOA Speer RK73H1ETTP1000F") (at 231.14 83.82 90) (unit 1)
     (in_bom yes) (on_board yes) (dnp no)
     (property "Reference" "R24" (at 224.79 82.55 90)
@@
     )
   )
-  (symbol (lib_id "Auto_Library_WUT:KOA Speer RK73H1ETTP1000F") (at 231.14 86.36 90) (unit 1)
+  (symbol (lib_id "Preferred_WUT:KOA Speer RK73H1ETTP1000F") (at 231.14 86.36 90) (unit 1)
     (in_bom yes) (on_board yes) (dnp no)
     (property "Reference" "R136" (at 224.79 85.09 90)
@@
     )
   )
-  (symbol (lib_id "Auto_Library_WUT:KOA Speer RK73H1ETTP1000F") (at 175.26 81.28 90) (unit 1)
+  (symbol (lib_id "Preferred_WUT:KOA Speer RK73H1ETTP1000F") (at 175.26 81.28 90) (unit 1)
     (in_bom yes) (on_board yes) (dnp no)
     (property "Reference" "R33" (at 168.91 80.01 90)
@@
     )
   )
-  (symbol (lib_id "Auto_Library_WUT:Lite-On_LTST-C193KRKT-5A ") (at 104.14 123.19 270) (unit 1)
+  (symbol (lib_id "Preferred_WUT:Lite-On_LTST-C193KRKT-5A ") (at 104.14 123.19 270) (unit 1)
     (in_bom yes) (on_board yes) (dnp no)
     (property "Reference" "LD1" (at 106.68 123.19 90)
@@
     )
   )
-  (symbol (lib_id "Auto_Library_WUT:KOA Speer RK73H1ETTP1001F") (at 255.27 149.86 270) (mirror x) (unit 1)
+  (symbol (lib_id "Preferred_WUT:KOA Speer RK73H1ETTP1001F") (at 255.27 149.86 270) (mirror x) (unit 1)
     (in_bom yes) (on_board yes) (dnp no) (fields_autoplaced)
     (property "Reference" "R54" (at 255.27 143.51 90)
@@
     )
   )
-  (symbol (lib_id "Auto_Library_WUT:KOA Speer RK73H1ETTP1000F") (at 175.26 83.82 90) (unit 1)
+  (symbol (lib_id "Preferred_WUT:KOA Speer RK73H1ETTP1000F") (at 175.26 83.82 90) (unit 1)
     (in_bom yes) (on_board yes) (dnp no)
     (property "Reference" "R34" (at 168.91 82.55 90)
@@
     )
   )
-  (symbol (lib_id "Auto_Library_WUT:KOA Speer RK73Z1ETTP") (at 175.26 123.19 90) (unit 1)
+  (symbol (lib_id "Preferred_WUT:KOA Speer RK73Z1ETTP") (at 175.26 123.19 90) (unit 1)
     (in_bom yes) (on_board yes) (dnp no)
     (property "Reference" "R52" (at 171.45 121.92 90)

Commit message: layout progress
Parts:
- removed R33, R34, R6, R9: 100R, Resistor_SMD:R_0402_1005Metric, symbol Preferred_WUT:KOA Speer RK73H1ETTP1000F
- added R12: 33R, Resistor_SMD:R_0402_1005Metric, symbol AAA_Preferred_WUT:KOA Speer RK73H1ETTP33R0F
- C3: renamed from C116; symbol Preferred_WUT:Yageo CC0402KRX7R8BB104 -> AAA_Preferred_WUT:Yageo CC0402KRX7R8BB104
- C6: renamed from C125; symbol Preferred_WUT:Yageo CC0402KRX7R8BB104 -> AAA_Preferred_WUT:Yageo CC0402KRX7R8BB104
- D12: renamed from D7; symbol Preferred_WUT:nexperia PESD3V3U1UB,115 -> AAA_Preferred_WUT:nexperia PESD3V3U1UB,115
- LD2: renamed from LD1; symbol Preferred_WUT:Lite-On_LTST-C193KRKT-5A -> AAA_Preferred_WUT:Lite-On_LTST-C193KRKT-5A
- LD3: symbol Preferred_WUT:Ekinglux_E6C0603VGAC1UDA -> AAA_Preferred_WUT:Ekinglux_E6C0603VGAC1UDA
- R13: renamed from R7; symbol Preferred_WUT:KOA Speer RK73H1ETTP33R0F -> AAA_Preferred_WUT:KOA Speer RK73H1ETTP33R0F
- R14: renamed from R53; symbol Preferred_WUT:KOA Speer RK73Z1ETTP -> AAA_Preferred_WUT:KOA Speer RK73Z1ETTP
- R15: renamed from R52; symbol Preferred_WUT:KOA Speer RK73Z1ETTP -> AAA_Preferred_WUT:KOA Speer RK73Z1ETTP
- R16: renamed from R60; symbol Preferred_WUT:KOA Speer RK73H1ETTP1000F -> AAA_Preferred_WUT:KOA Speer RK73H1ETTP1000F
- R18: renamed from R5; symbol Preferred_WUT:KOA Speer RK73H1ETTP1000F -> AAA_Preferred_WUT:KOA Speer RK73H1ETTP1000F
- R19: renamed from R37; symbol Preferred_WUT:KOA Speer RK73H1ETTP1000F -> AAA_Preferred_WUT:KOA Speer RK73H1ETTP1000F
- R20: renamed from R36; symbol Preferred_WUT:KOA Speer RK73H1ETTP1000F -> AAA_Preferred_WUT:KOA Speer RK73H1ETTP1000F
- R21: renamed from R8; symbol Preferred_WUT:KOA Speer RK73H1ETTP1000F -> AAA_Preferred_WUT:KOA Speer RK73H1ETTP1000F
- R22: renamed from R14; symbol Preferred_WUT:KOA Speer RK73H1ETTP1000F -> AAA_Preferred_WUT:KOA Speer RK73H1ETTP1000F
- R23: renamed from R24; symbol Preferred_WUT:KOA Speer RK73H1ETTP1000F -> AAA_Preferred_WUT:KOA Speer RK73H1ETTP1000F
- R24: renamed from R136; symbol Preferred_WUT:KOA Speer RK73H1ETTP1000F -> AAA_Preferred_WUT:KOA Speer RK73H1ETTP1000F
- R25: renamed from R56; symbol Preferred_WUT:KOA Speer RK73Z1ETTP -> AAA_Preferred_WUT:KOA Speer RK73Z1ETTP
- R27: renamed from R54; symbol Preferred_WUT:KOA Speer RK73H1ETTP1001F -> AAA_Preferred_WUT:KOA Speer RK73H1ETTP1001F
- R6: renamed from R55; symbol Preferred_WUT:KOA Speer RK73H1ETTP1001F -> AAA_Preferred_WUT:KOA Speer RK73H1ETTP1001F
- renumbered C123 to C4, C124 to C5, C158 to C7, CN13 to CN3, R32 to R10, R117 to R11, R4 to R17, R35 to R26, R15 to R28, R130 to R29, R131 to R30, R2 to R7, R3 to R8, R31 to R9, U8 to U3
Connections:
- net COMMS_GREEN: now also CN4.44 (GPIO10)
- net COMMS_RED: now also R12.2
- net STATUS_GREEN: now also CN4.31 (GPIO12)
- net STATUS_RED: now also CN4.28 (GPIO13)
- net at CN4.38 (GPIO11): now also R12.1
Other:
- note removed: "For PWM on GPIO12 and GPIO13, see https://pypi.org/project/rpi-hardware-pwm/"
- note removed: "See https://forums.raspberrypi.com/viewtopic.php?t=302634 for use of GPIO as second SDIO interface"
- moved on the sheet: R11, R17
