File: Master Timing Card.kicad_sch (KiCad schematic)
At the start: 13 parts, among them CN1 Pin_03, CN2 Samtec GRF1-J-P-08-E-RA-TH1, CN3 Amphenol 86093488613755E1LF, U1 Microchip 24LC024-E/MC, U2 Analog MAX3483ESA+

Commit message: Added ESD and tided up PSU
Other:
- added sheet Power Supplies (power.kicad_sch)
Changed lines of the file:
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@@
     )
   )
-  (sheet (at 195.58 267.97) (size 44.45 16.51) (fields_autoplaced)
+  (sheet (at 66.04 262.89) (size 44.45 16.51) (fields_autoplaced)
     (stroke (width 0.1524) (type solid))
     (fill (color 0 0 0 0.0000))
-    (property "Sheetname" "CM4 Interfaces" (at 195.58 267.2584 0)
+    (property "Sheetname" "CM4 Interfaces" (at 66.04 262.1784 0)
       (effects (font (size 1.27 1.27)) (justify left bottom))
     )
-    (property "Sheetfile" "cm4_io.kicad_sch" (at 195.58 285.0646 0)
+    (property "Sheetfile" "cm4_io.kicad_sch" (at 66.04 279.9846 0)
       (effects (font (size 1.27 1.27)) (justify left top))
     )
@@
       )
     )
+  )
+  (sheet (at 119.38 262.89) (size 44.45 16.51) (fields_autoplaced)
+    (stroke (width 0.1524) (type solid))
+    (fill (color 0 0 0 0.0000))
+    (property "Sheetname" "Power Supplies" (at 119.38 262.1784 0)
+      (effects (font (size 1.27 1.27)) (justify left bottom))
+    )
+    (property "Sheetfile" "power.kicad_sch" (at 119.38 279.9846 0)
+      (effects (font (size 1.27 1.27)) (justify left top))
+    )
+    (property "Field2" "" (at 119.38 262.89 0)
+      (effects (font (size 1.27 1.27)) hide)
+    )
+    (instances
+      (project "Master Timing Card"
+        (path "/6e8e281e-e30f-459d-852f-231836068db5" (page "9"))
+      )
+    )

Commit message: Schematic mostly done
Parts:
- added D10, D11, D12, D13, D14, D15, D16, D17: 5V0, Diode_SMD:D_SOD-523, symbol Auto_Library_WUT:Littelfuse AQ3522-01LTG
- added LD9: WP130WCP_2EGW, LED_WUT:Kingbright_WP130WCP_2EGW, symbol LED_WUT:Kingbright_WP130WCP_2EGW
- added R10, R11, R12, R13: 1k0, Resistor_SMD:R_0402_1005Metric, symbol Auto_Library_WUT:KOA Speer RK73H1ETTP1001F
- added R132: 100R, Resistor_SMD:R_0402_1005Metric, symbol Auto_Library_WUT:KOA Speer RK73H1ETTP1000F
- CN1: value Pin_03 -> M20-9990346
Connections:
- net 0V: now also D10.2 (A), D11.2 (A), D12.2 (A), D13.2 (A), D14.2 (A), D15.2 (A), D16.2 (A), D17.2 (A), LD9.2, LD9.5
- net PSU_EEPROM_3V3: now also R132.2
- net at C3.1, FB1.2, U1.8 (VCC): no longer CN1.1 (Pin_1)
- net RF1: now reaches CN2.1 (In)
- net RF1: now also D17.1 (K)
- net RF2: now reaches CN2.2 (In)
- net RF2: now also D16.1 (K)
- net RF3: now reaches CN2.3 (In)
- net RF3: now also D15.1 (K)
- net RF4: now reaches CN2.4 (In)
- net RF4: now also D14.1 (K)
- net RF5: now reaches CN2.5 (In)
- net RF5: now also D13.1 (K)
- net RF6: now reaches CN2.6 (In)
- net RF6: now also D12.1 (K)
- net RF7: now reaches CN2.7 (In)
- net RF7: now also D11.1 (K)
- net RF8: now reaches CN2.8 (In)
- net RF8: now also D10.1 (K)
- removed net +12V: CN3.a7, CN3.a8, CN3.b7, CN3.b8, CN3.c7, CN3.c8
- removed net +24V: CN3.a4, CN3.a5, CN3.b4, CN3.b5, CN3.c4, CN3.c5
- net +3.3V renamed 3V3
- removed net +48V: CN3.a1, CN3.a2, CN3.b1, CN3.b2, CN3.c1, CN3.c2
- net RX renamed RS485_RX
- net TX renamed RS485_TX
- net ~{R}/W renamed RS485_~{R}/W
- new net: CN3.a1, CN3.a2
- new net: CN3.a4, CN3.a5
- new net: CN3.a7, CN3.a8
- new net: CN3.c1, CN3.c2
- new net: CN3.c4, CN3.c5
- new net: CN3.c7, CN3.c8
- new net: CN3.b4, CN3.b5
- new net: CN3.b7, CN3.b8
- new net: LD9.3, R12.2
- new net: LD9.1, R13.2
- new net: LD9.4, R10.2
- new net: LD9.6, R11.2
- new net: CN1.1 (Pin_1), R132.1
- new net Pi CM4 - GPIO/COMMS_GREEN: R11.1
- new net Pi CM4 - GPIO/COMMS_RED: R10.1
- new net Pi CM4 - GPIO/STATUS_GREEN: R12.1
- new net Pi CM4 - GPIO/STATUS_RED: R13.1
Other:
- sheet CM4 Interfaces ports: added PTP_PPS; removed none
- sheet GPS ports: added GNSS_25MHZ, GNSS_PPS, GNSS_RESET, GNSS_RX, GNSS_TX, PTP_PPS; removed none
- sheet PLL and SFP ports: added PLL1_SCL, PLL1_SDA, PLL2_SCL, PLL2_SDA, PLL_LOCK, PLL_OE, RF1, RF2, RF3, RF4, RF5, RF6, RF7, RF8, SFP_LOS_OD, SFP_SCL, SFP_SDA, SFP_TX_DISABLE, SFP_TX_FAULT_OD, ~{SFP_PRESENT}; removed none
- sheet Pi CM4 - GPIO ports: added 3V3_PCIE_EN, 3V3_SENSE_N, 3V3_SENSE_P, COMMS_GREEN, COMMS_RED, GNSS_PPS, GNSS_RESET, PCIE_PWR_GOOD, PLL1_SCL, PLL1_SDA, PLL2_SCL, PLL2_SDA, PLL_LOCK, PLL_OE, PWR_CRITICAL, RS485_~{RX}/TX, SFP_LOS, SFP_TX_DISABLE, SFP_TX_FAULT, STATUS_GREEN, STATUS_RED, UART0_RX, UART0_TX, UART3_RX, UART3_TX, ~{SFP_PRESENT}; removed none
- sheet Power Supplies ports: added 3V3_PCIE_EN, PCIE_PGOOD, POWER_CRITICAL, POWER_SENSE3_N, POWER_SENSE3_P, SCL, SDA; removed none
- note added: "Raspberry Pi CM4"
- note added: "TODO Backplane Connector pinout"
- moved on the sheet: C1, C2, C3, CN1, CN2, FB1, LAYOUT1, LAYOUT2, LAYOUT3, R1, U1, U2

Commit message: schematic complete
Parts:
- removed C3: 100n, Capacitor_SMD:C_0402_1005Metric, symbol Auto_Library_WUT:Yageo CC0402KRX7R8BB104
- removed CN1: M20-9990346, Connector_PinHeader_2.54mm:PinHeader_1x03_P2.54mm_Vertical, symbol Connector_WUT:Harwin_M20-9990346
- removed FB1: 1k8, Inductor_SMD:L_0402_1005Metric, symbol Auto_Library_WUT:Murata BLM15BD182SN1D
- removed R132: 100R, Resistor_SMD:R_0402_1005Metric, symbol Auto_Library_WUT:KOA Speer RK73H1ETTP1000F
- removed U1: Microchip 24LC024-E/MC, Package_DFN_QFN:DFN-8-1EP_3x2mm_P0.5mm_EP1.36x1.46mm, symbol IC_WUT:24LC024-E/MC
- added U1: DS2431P+, Package_SO_J-Lead:TSOC-6_3.76x3.94mm_P1.27mm, symbol IC_WUT:Analog_DS2431P+
Connections:
- net PSU_EEPROM_ADDR2 is gone; now on net 0V: CN3.a16
- net 0V: now also U1.1 (GND); no longer CN3.a10, CN3.a3, CN3.a6, CN3.a9, CN3.b10, CN3.b3, CN3.b6, CN3.b9, CN3.c10, CN3.c3, CN3.c6, CN3.c9
- net RS485_A: now also CN3.b1; no longer CN3.c14
- net RS485_B: now also CN3.a1; no longer CN3.c13
- net at CN3.a2: no longer CN3.a1
- net at CN3.a4: no longer CN3.a5
- net at CN3.a7: no longer CN3.a8
- net at CN3.c1: now also U1.2 (IO); no longer CN3.c2
- net at CN3.c4: no longer CN3.c5
- net at CN3.c7: no longer CN3.c8
- net at CN3.b4: no longer CN3.b5
- net at CN3.b7: no longer CN3.b8
- net PSU_EEPROM_3V3: no longer names the net of CN3.c15
- net PSU_EEPROM_ADDR0: no longer names the net of CN3.c16
- net PSU_EEPROM_ADDR1: no longer names the net of CN3.b16
- net PSU_EEPROM_SCL: no longer names the net of CN3.b15
- net PSU_EEPROM_SDA: no longer names the net of CN3.a15
- net SLOTS_EEPROM_3V3: no longer names the net of CN3.a13
- net SLOTS_EEPROM_SCL: no longer names the net of CN3.b14
- net SLOTS_EEPROM_SDA: no longer names the net of CN3.b13
- net SLOTS_EEPROM_WP: no longer names the net of CN3.a14
- no-connect marks 0 -> 44
Other:
- sheet GPS ports: added CLK_SEL, REF_CLK_N, REF_CLK_P; removed GNSS_25MHZ
- sheet PLL and SFP ports: added CLK_SEL, REF_CLK_N, REF_CLK_P; removed none
- sheet Pi CM4 - GPIO ports: added PLL_CLK_SEL, REF_CLK_SEL; removed none
- note added: "I2C Addresses: SFP: 0x50 INA3221: 0x40 RC32504: 0x09"
- moved on the sheet: CN3A, CN3B, CN3C

Commit message: Moved to preferred library
Parts:
- C1: symbol Auto_Library_WUT:Samsung Electro-Mechanics CL10A106MO8NQNC -> Preferred_WUT:Samsung Electro-Mechanics CL10A106MO8NQNC
- C2: symbol Auto_Library_WUT:Yageo CC0402KRX7R8BB104 -> Preferred_WUT:Yageo CC0402KRX7R8BB104
- D10, D11, D12, D13, D14, D15, D16, D17: symbol Auto_Library_WUT:Littelfuse AQ3522-01LTG -> Preferred_WUT:Littelfuse AQ3522-01LTG
- R10, R11, R12, R13: symbol Auto_Library_WUT:KOA Speer RK73H1ETTP1001F -> Preferred_WUT:KOA Speer RK73H1ETTP1001F
Changed lines of the file:
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@@
     )
   )
-  (symbol (lib_id "Auto_Library_WUT:Littelfuse AQ3522-01LTG") (at 339.09 241.3 90) (unit 1)
+  (symbol (lib_id "Preferred_WUT:Littelfuse AQ3522-01LTG") (at 339.09 241.3 90) (unit 1)
     (in_bom yes) (on_board yes) (dnp no) (fields_autoplaced)
     (property "Reference" "D11" (at 341.63 239.776 90)
@@
     )
   )
-  (symbol (lib_id "Auto_Library_WUT:KOA Speer RK73H1ETTP1001F") (at 193.04 219.71 90) (unit 1)
+  (symbol (lib_id "Preferred_WUT:KOA Speer RK73H1ETTP1001F") (at 193.04 219.71 90) (unit 1)
     (in_bom yes) (on_board yes) (dnp no)
     (property "Reference" "R12" (at 189.23 218.44 90) (do_not_autoplace)
@@
     )
   )
-  (symbol (lib_id "Auto_Library_WUT:Littelfuse AQ3522-01LTG") (at 285.75 241.3 90) (unit 1)
+  (symbol (lib_id "Preferred_WUT:Littelfuse AQ3522-01LTG") (at 285.75 241.3 90) (unit 1)
     (in_bom yes) (on_board yes) (dnp no) (fields_autoplaced)
     (property "Reference" "D17" (at 288.29 239.776 90)
@@
     )
   )
-  (symbol (lib_id "Auto_Library_WUT:Littelfuse AQ3522-01LTG") (at 330.2 241.3 90) (unit 1)
+  (symbol (lib_id "Preferred_WUT:Littelfuse AQ3522-01LTG") (at 330.2 241.3 90) (unit 1)
     (in_bom yes) (on_board yes) (dnp no) (fields_autoplaced)
     (property "Reference" "D12" (at 332.74 239.776 90)
@@
     )
   )
-  (symbol (lib_id "Auto_Library_WUT:Littelfuse AQ3522-01LTG") (at 312.42 241.3 90) (unit 1)
+  (symbol (lib_id "Preferred_WUT:Littelfuse AQ3522-01LTG") (at 312.42 241.3 90) (unit 1)
     (in_bom yes) (on_board yes) (dnp no) (fields_autoplaced)
     (property "Reference" "D14" (at 314.96 239.776 90)
@@
     )
   )
-  (symbol (lib_id "Auto_Library_WUT:Samsung Electro-Mechanics CL10A106MO8NQNC") (at 264.16 55.88 0) (unit 1)
+  (symbol (lib_id "Preferred_WUT:Samsung Electro-Mechanics CL10A106MO8NQNC") (at 264.16 55.88 0) (unit 1)
     (in_bom yes) (on_board yes) (dnp no) (fields_autoplaced)
     (property "Reference" "C1" (at 266.7 53.34 0) (do_not_autoplace)
@@
     )
   )
-  (symbol (lib_id "Auto_Library_WUT:Littelfuse AQ3522-01LTG") (at 294.64 241.3 90) (unit 1)
+  (symbol (lib_id "Preferred_WUT:Littelfuse AQ3522-01LTG") (at 294.64 241.3 90) (unit 1)
     (in_bom yes) (on_board yes) (dnp no) (fields_autoplaced)
     (property "Reference" "D16" (at 297.18 239.776 90)
@@
     )
   )
-  (symbol (lib_id "Auto_Library_WUT:Yageo CC0402KRX7R8BB104") (at 278.13 55.88 0) (unit 1)
+  (symbol (lib_id "Preferred_WUT:Yageo CC0402KRX7R8BB104") (at 278.13 55.88 0) (unit 1)
     (in_bom yes) (on_board yes) (dnp no) (fields_autoplaced)
     (property "Reference" "C2" (at 280.67 53.34 0) (do_not_autoplace)
@@
     )
   )
-  (symbol (lib_id "Auto_Library_WUT:Littelfuse AQ3522-01LTG") (at 347.98 241.3 90) (unit 1)
+  (symbol (lib_id "Preferred_WUT:Littelfuse AQ3522-01LTG") (at 347.98 241.3 90) (unit 1)
     (in_bom yes) (on_board yes) (dnp no) (fields_autoplaced)
     (property "Reference" "D10" (at 350.52 239.776 90)
@@
     )
   )
-  (symbol (lib_id "Auto_Library_WUT:Littelfuse AQ3522-01LTG") (at 303.53 241.3 90) (unit 1)
+  (symbol (lib_id "Preferred_WUT:Littelfuse AQ3522-01LTG") (at 303.53 241.3 90) (unit 1)
     (in_bom yes) (on_board yes) (dnp no) (fields_autoplaced)
     (property "Reference" "D15" (at 306.07 239.776 90)
@@
     )
   )
-  (symbol (lib_id "Auto_Library_WUT:Littelfuse AQ3522-01LTG") (at 321.31 241.3 90) (unit 1)
+  (symbol (lib_id "Preferred_WUT:Littelfuse AQ3522-01LTG") (at 321.31 241.3 90) (unit 1)
     (in_bom yes) (on_board yes) (dnp no) (fields_autoplaced)
     (property "Reference" "D13" (at 323.85 239.776 90)
@@
     )
   )
-  (symbol (lib_id "Auto_Library_WUT:KOA Speer RK73H1ETTP1001F") (at 193.04 227.33 90) (unit 1)
+  (symbol (lib_id "Preferred_WUT:KOA Speer RK73H1ETTP1001F") (at 193.04 227.33 90) (unit 1)
     (in_bom yes) (on_board yes) (dnp no)
     (property "Reference" "R10" (at 189.23 226.06 90) (do_not_autoplace)
@@
     )
   )
-  (symbol (lib_id "Auto_Library_WUT:KOA Speer RK73H1ETTP1001F") (at 193.04 232.41 90) (unit 1)
+  (symbol (lib_id "Preferred_WUT:KOA Speer RK73H1ETTP1001F") (at 193.04 232.41 90) (unit 1)
     (in_bom yes) (on_board yes) (dnp no)
     (property "Reference" "R11" (at 189.23 231.14 90) (do_not_autoplace)
@@
     )
   )
-  (symbol (lib_id "Auto_Library_WUT:KOA Speer RK73H1ETTP1001F") (at 193.04 214.63 90) (unit 1)
+  (symbol (lib_id "Preferred_WUT:KOA Speer RK73H1ETTP1001F") (at 193.04 214.63 90) (unit 1)
     (in_bom yes) (on_board yes) (dnp no)
     (property "Reference" "R13" (at 189.23 213.36 90) (do_not_autoplace)

Commit message: Started placement
Parts:
- added H8: ~, Misc_WUT:Logo_10mmx10mm, symbol Layout_WUT:Logo_10mmx10mm
Changed lines of the file:
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@@
+    )
+  )
+  (symbol (lib_id "Layout_WUT:Logo_10mmx10mm") (at 219.71 271.78 0) (unit 1)
+    (in_bom no) (on_board yes) (dnp no) (fields_autoplaced)
+    (property "Reference" "H8" (at 228.6 271.78 0)
+      (effects (font (size 1.27 1.27)) (justify left))
+    )
+    (property "Value" "~" (at 219.71 271.78 0)
+      (effects (font (size 1.27 1.27)))
+    )
+    (property "Footprint" "Misc_WUT:Logo_10mmx10mm" (at 219.71 271.78 0)
+      (effects (font (size 1.27 1.27)) hide)
+    )
+    (property "Datasheet" "" (at 219.71 271.78 0)
+      (effects (font (size 1.27 1.27)) hide)
+    )
+    (instances
+      (project "Master Timing Card"
+        (path "/6e8e281e-e30f-459d-852f-231836068db5"
+          (reference "H8") (unit 1)
+        )
+      )
     )
   )

Commit message: layout progress
Parts:
- added D10, D6, D9: 3V3, Diode_SMD:D_SOD-523, symbol AAA_Preferred_WUT:nexperia PESD3V3U1UB,115
- C1: symbol Preferred_WUT:Samsung Electro-Mechanics CL10A106MO8NQNC -> AAA_Preferred_WUT:Samsung Electro-Mechanics CL10A106MO8NQNC
- C2: symbol Preferred_WUT:Yageo CC0402KRX7R8BB104 -> AAA_Preferred_WUT:Yageo CC0402KRX7R8BB104
- D1: renamed from D17; symbol Preferred_WUT:Littelfuse AQ3522-01LTG -> AAA_Preferred_WUT:Littelfuse AQ3522-01LTG
- D11: renamed from D10; symbol Preferred_WUT:Littelfuse AQ3522-01LTG -> AAA_Preferred_WUT:Littelfuse AQ3522-01LTG
- D2: renamed from D16; symbol Preferred_WUT:Littelfuse AQ3522-01LTG -> AAA_Preferred_WUT:Littelfuse AQ3522-01LTG
- D3: renamed from D15; symbol Preferred_WUT:Littelfuse AQ3522-01LTG -> AAA_Preferred_WUT:Littelfuse AQ3522-01LTG
- D4: renamed from D14; symbol Preferred_WUT:Littelfuse AQ3522-01LTG -> AAA_Preferred_WUT:Littelfuse AQ3522-01LTG
- D5: renamed from D13; symbol Preferred_WUT:Littelfuse AQ3522-01LTG -> AAA_Preferred_WUT:Littelfuse AQ3522-01LTG
- D7: renamed from D12; symbol Preferred_WUT:Littelfuse AQ3522-01LTG -> AAA_Preferred_WUT:Littelfuse AQ3522-01LTG
- D8: renamed from D11; symbol Preferred_WUT:Littelfuse AQ3522-01LTG -> AAA_Preferred_WUT:Littelfuse AQ3522-01LTG
- R1: renamed from R13; symbol Preferred_WUT:KOA Speer RK73H1ETTP1001F -> AAA_Preferred_WUT:KOA Speer RK73H1ETTP1001F
- R2: renamed from R12; symbol Preferred_WUT:KOA Speer RK73H1ETTP1001F -> AAA_Preferred_WUT:KOA Speer RK73H1ETTP1001F
- R3: renamed from R10; symbol Preferred_WUT:KOA Speer RK73H1ETTP1001F -> AAA_Preferred_WUT:KOA Speer RK73H1ETTP1001F
- R4: renamed from R11; symbol Preferred_WUT:KOA Speer RK73H1ETTP1001F -> AAA_Preferred_WUT:KOA Speer RK73H1ETTP1001F
- renumbered CN2 to CN1, CN3 to CN2, H8 to H1, LD9 to LD1, R1 to R5, U2 to U1, U1 to U2
Connections:
- net 0V: now also D10.2 (A), D6.2 (A), D9.2 (A)
- net RS485_A: now also D9.1 (K)
- net RS485_B: now also D10.1 (K)
- net at CN2.c1, U2.2 (IO): now also D6.1 (K)

Commit message: getting there
Changed lines of the file:
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@@
   (junction (at 347.98 233.68) (diameter 0) (color 0 0 0 0)
   )
-  (junction (at 176.53 125.73) (diameter 0) (color 0 0 0 0)
-  )
   (junction (at 373.38 213.36) (diameter 0) (color 0 0 0 0)
   )
+  (junction (at 373.38 223.52) (diameter 0) (color 0 0 0 0)
+  )
+  (junction (at 311.15 66.04) (diameter 0.9144) (color 0 0 0 0)
+  )
+  (junction (at 222.25 229.87) (diameter 0) (color 0 0 0 0)
+  )
+  (junction (at 279.4 72.39) (diameter 0.9144) (color 0 0 0 0)
+  )
+  (junction (at 373.38 208.28) (diameter 0) (color 0 0 0 0)
+  )
+  (junction (at 285.75 198.12) (diameter 0) (color 0 0 0 0)
+  )
+  (junction (at 278.13 49.53) (diameter 0.9144) (color 0 0 0 0)
+  )
+  (junction (at 346.71 91.44) (diameter 0) (color 0 0 0 0)
+  )
+  (junction (at 339.09 228.6) (diameter 0) (color 0 0 0 0)
+  )
+  (junction (at 326.39 147.32) (diameter 0) (color 0 0 0 0)
+  )
+  (junction (at 373.38 203.2) (diameter 0) (color 0 0 0 0)
+  )
+  (junction (at 311.15 81.28) (diameter 0.9144) (color 0 0 0 0)
+  )
+  (junction (at 312.42 213.36) (diameter 0) (color 0 0 0 0)
+  )
+  (junction (at 303.53 208.28) (diameter 0) (color 0 0 0 0)
+  )
+  (junction (at 173.99 120.65) (diameter 0) (color 0 0 0 0)
+  )
+  (junction (at 373.38 233.68) (diameter 0) (color 0 0 0 0)
+  )
+  (junction (at 347.98 35.56) (diameter 0) (color 0 0 0 0)
+  )
+  (junction (at 294.64 203.2) (diameter 0) (color 0 0 0 0)
+  )
+  (junction (at 330.2 223.52) (diameter 0) (color 0 0 0 0)
+  )
+  (junction (at 321.31 218.44) (diameter 0) (color 0 0 0 0)
+  )
+  (junction (at 264.16 49.53) (diameter 0.9144) (color 0 0 0 0)
+  )
   (junction (at 173.99 143.51) (diameter 0) (color 0 0 0 0)
   )
-  (junction (at 373.38 223.52) (diameter 0) (color 0 0 0 0)
-  )
-  (junction (at 311.15 66.04) (diameter 0.9144) (color 0 0 0 0)
-  )
-  (junction (at 222.25 229.87) (diameter 0) (color 0 0 0 0)
-  )
-  (junction (at 279.4 72.39) (diameter 0.9144) (color 0 0 0 0)
-  )
-  (junction (at 373.38 208.28) (diameter 0) (color 0 0 0 0)
-  )
-  (junction (at 285.75 198.12) (diameter 0) (color 0 0 0 0)
-  )
-  (junction (at 278.13 49.53) (diameter 0.9144) (color 0 0 0 0)
-  )
-  (junction (at 346.71 91.44) (diameter 0) (color 0 0 0 0)
-  )
-  (junction (at 339.09 228.6) (diameter 0) (color 0 0 0 0)
-  )
-  (junction (at 326.39 147.32) (diameter 0) (color 0 0 0 0)
+  (junction (at 373.38 218.44) (diameter 0) (color 0 0 0 0)
+  )
+  (junction (at 176.53 118.11) (diameter 0) (color 0 0 0 0)
   )
   (junction (at 176.53 140.97) (diameter 0) (color 0 0 0 0)
-  )
-  (junction (at 373.38 203.2) (diameter 0) (color 0 0 0 0)
-  )
-  (junction (at 311.15 81.28) (diameter 0.9144) (color 0 0 0 0)
-  )
-  (junction (at 312.42 213.36) (diameter 0) (color 0 0 0 0)
-  )
-  (junction (at 303.53 208.28) (diameter 0) (color 0 0 0 0)
-  )
-  (junction (at 373.38 233.68) (diameter 0) (color 0 0 0 0)
-  )
-  (junction (at 347.98 35.56) (diameter 0) (color 0 0 0 0)
-  )
-  (junction (at 173.99 128.27) (diameter 0) (color 0 0 0 0)
-  )
-  (junction (at 294.64 203.2) (diameter 0) (color 0 0 0 0)
-  )
-  (junction (at 330.2 223.52) (diameter 0) (color 0 0 0 0)
-  )
-  (junction (at 321.31 218.44) (diameter 0) (color 0 0 0 0)
-  )
-  (junction (at 264.16 49.53) (diameter 0.9144) (color 0 0 0 0)
-  )
-  (junction (at 373.38 218.44) (diameter 0) (color 0 0 0 0)
   )
   (no_connect (at 358.14 154.94))
@@
     (stroke (width 0) (type default))
   )
-  (wire (pts (xy 173.99 128.27) (xy 173.99 143.51))
-    (stroke (width 0) (type default))
-  )
   (wire (pts (xy 147.32 227.33) (xy 189.23 227.33))
     (stroke (width 0) (type default))
@@
     (stroke (width 0) (type default))
   )
-  (wire (pts (xy 176.53 125.73) (xy 185.42 125.73))
+  (wire (pts (xy 147.32 125.73) (xy 185.42 125.73))
     (stroke (width 0) (type default))
   )
@@
     (stroke (width 0) (type default))
   )
-  (wire (pts (xy 147.32 120.65) (xy 185.42 120.65))
+  (wire (pts (xy 147.32 120.65) (xy 173.99 120.65))
     (stroke (width 0) (type default))
   )
@@
     (stroke (width 0) (type default))
   )
+  (wire (pts (xy 173.99 120.65) (xy 173.99 143.51))
+    (stroke (width 0) (type default))
+  )
   (wire (pts (xy 294.64 245.11) (xy 294.64 247.65))
     (stroke (width 0) (type default))
@@
     (stroke (width 0) (type default))
   )
-  (wire (pts (xy 147.32 125.73) (xy 176.53 125.73))
-    (stroke (width 0) (type default))
-  )
   (wire (pts (xy 247.65 130.81) (xy 259.08 130.81))
     (stroke (width 0) (type default))
@@
     (stroke (width 0) (type solid))
   )
+  (wire (pts (xy 173.99 120.65) (xy 185.42 120.65))
+    (stroke (width 0) (type default))
+  )
   (wire (pts (xy 275.59 228.6) (xy 339.09 228.6))
     (stroke (width 0) (type default))
@@
     (stroke (width 0) (type default))
   )
+  (wire (pts (xy 176.53 118.11) (xy 185.42 118.11))
+    (stroke (width 0) (type default))
+  )
   (wire (pts (xy 347.98 35.56) (xy 358.14 35.56))
     (stroke (width 0) (type default))
@@
     (stroke (width 0) (type default))
   )
-  (wire (pts (xy 176.53 140.97) (xy 176.53 125.73))
-    (stroke (width 0) (type default))
-  )
   (wire (pts (xy 344.17 91.44) (xy 346.71 91.44))
     (stroke (width 0) (type default))
@@
     (stroke (width 0) (type default))
   )
-  (wire (pts (xy 147.32 128.27) (xy 173.99 128.27))
-    (stroke (width 0) (type default))
-  )
   (wire (pts (xy 196.85 232.41) (xy 204.47 232.41))
     (stroke (width 0) (type default))
@@
     (stroke (width 0) (type default))
   )
+  (wire (pts (xy 176.53 118.11) (xy 176.53 140.97))
+    (stroke (width 0) (type default))
+  )
   (wire (pts (xy 196.85 219.71) (xy 204.47 219.71))
     (stroke (width 0) (type default))
@@
     (stroke (width 0) (type default))
   )
-  (wire (pts (xy 173.99 128.27) (xy 185.42 128.27))
+  (wire (pts (xy 147.32 128.27) (xy 185.42 128.27))
     (stroke (width 0) (type default))
   )
@@
     (stroke (width 0) (type default))
   )
-  (wire (pts (xy 147.32 118.11) (xy 185.42 118.11))
-    (stroke (width 0) (type default))
-  )
+  (wire (pts (xy 147.32 118.11) (xy 176.53 118.11))
+    (stroke (width 0) (type default))
+  )
