File: Master Timing Card.kicad_sch (KiCad schematic)
At the start: 27 parts, among them CN1 Samtec GRF1-J-P-08-E-RA-TH1, CN2 Amphenol 86093488613755E1LF, U1 Analog MAX3483ESA+, U2 DS2431P+

Commit message: committing before attempting scripting
Changed lines of the file:
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@@
   (junction (at 373.38 208.28) (diameter 0) (color 0 0 0 0)
   )
+  (junction (at 179.07 128.27) (diameter 0) (color 0 0 0 0)
+  )
   (junction (at 285.75 198.12) (diameter 0) (color 0 0 0 0)
   )
@@
   (junction (at 264.16 49.53) (diameter 0.9144) (color 0 0 0 0)
   )
-  (junction (at 173.99 143.51) (diameter 0) (color 0 0 0 0)
-  )
   (junction (at 373.38 218.44) (diameter 0) (color 0 0 0 0)
   )
   (junction (at 176.53 118.11) (diameter 0) (color 0 0 0 0)
   )
-  (junction (at 176.53 140.97) (diameter 0) (color 0 0 0 0)
+  (junction (at 181.61 125.73) (diameter 0) (color 0 0 0 0)
   )
   (no_connect (at 358.14 154.94))
@@
     (stroke (width 0) (type default))
   )
-  (wire (pts (xy 173.99 143.51) (xy 173.99 171.45))
-    (stroke (width 0) (type default))
-  )
   (wire (pts (xy 147.32 181.61) (xy 185.42 181.61))
     (stroke (width 0) (type default))
@@
     (stroke (width 0) (type default))
   )
-  (wire (pts (xy 185.42 143.51) (xy 173.99 143.51))
-    (stroke (width 0) (type default))
-  )
-  (wire (pts (xy 147.32 125.73) (xy 185.42 125.73))
+  (wire (pts (xy 147.32 125.73) (xy 181.61 125.73))
     (stroke (width 0) (type default))
   )
@@
     (stroke (width 0) (type default))
   )
+  (wire (pts (xy 181.61 140.97) (xy 181.61 125.73))
+    (stroke (width 0) (type default))
+  )
   (wire (pts (xy 250.19 82.55) (xy 247.65 82.55))
     (stroke (width 0) (type default))
@@
     (stroke (width 0) (type default))
   )
-  (wire (pts (xy 173.99 120.65) (xy 173.99 143.51))
+  (wire (pts (xy 181.61 125.73) (xy 185.42 125.73))
+    (stroke (width 0) (type default))
+  )
+  (wire (pts (xy 173.99 120.65) (xy 173.99 171.45))
+    (stroke (width 0) (type default))
+  )
+  (wire (pts (xy 179.07 128.27) (xy 185.42 128.27))
     (stroke (width 0) (type default))
   )
@@
     (stroke (width 0) (type solid))
   )
-  (wire (pts (xy 185.42 140.97) (xy 176.53 140.97))
-    (stroke (width 0) (type default))
-  )
   (wire (pts (xy 281.94 72.39) (xy 279.4 72.39))
     (stroke (width 0) (type solid))
@@
     (stroke (width 0) (type default))
   )
+  (wire (pts (xy 179.07 143.51) (xy 179.07 128.27))
+    (stroke (width 0) (type default))
+  )
   (wire (pts (xy 294.64 203.2) (xy 353.06 203.2))
     (stroke (width 0) (type default))
@@
     (stroke (width 0) (type solid))
   )
+  (wire (pts (xy 185.42 143.51) (xy 179.07 143.51))
+    (stroke (width 0) (type default))
+  )
   (wire (pts (xy 285.75 245.11) (xy 285.75 247.65))
     (stroke (width 0) (type default))
@@
     (stroke (width 0) (type default))
   )
-  (wire (pts (xy 176.53 118.11) (xy 176.53 140.97))
+  (wire (pts (xy 176.53 118.11) (xy 176.53 168.91))
     (stroke (width 0) (type default))
   )
@@
     (stroke (width 0) (type default))
   )
+  (wire (pts (xy 185.42 140.97) (xy 181.61 140.97))
+    (stroke (width 0) (type default))
+  )
   (wire (pts (xy 264.16 59.69) (xy 264.16 62.23))
     (stroke (width 0) (type solid))
@@
     (stroke (width 0) (type default))
   )
-  (wire (pts (xy 147.32 128.27) (xy 185.42 128.27))
+  (wire (pts (xy 147.32 128.27) (xy 179.07 128.27))
     (stroke (width 0) (type default))
   )
@@
     (stroke (width 0) (type default))
   )
-  (wire (pts (xy 176.53 168.91) (xy 176.53 140.97))
-    (stroke (width 0) (type default))
-  )
