File: Master Timing Card.kicad_sch (KiCad schematic)
At the start: 28 parts, among them CN1 Samtec GRF1-J-P-08-E-RA-TH1, CN2 Amphenol 86093488613755E1LF, U1 Analog MAX3483ESA+, U2 DS2431P+

Commit message: released version
Connections:
- net 0V: now also CN2.a9, CN2.b9, CN2.c9
- net 12V: now reaches CN2.a8
- net 12V: now also CN2.b8, CN2.c8
- no-connect marks 43 -> 37
Other:
- note removed: "TODO Backplane Connector pinout"
Changed lines of the file:
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@@
   (no_connect (at 358.14 177.8))
   (no_connect (at 358.14 127))
-  (no_connect (at 358.14 165.1))
-  (no_connect (at 358.14 167.64))
   (no_connect (at 358.14 93.98))
   (no_connect (at 358.14 66.04))
@@
   (no_connect (at 358.14 121.92))
   (no_connect (at 358.14 114.3))
-  (no_connect (at 358.14 111.76))
   (no_connect (at 358.14 180.34))
   (no_connect (at 358.14 58.42))
-  (no_connect (at 358.14 55.88))
   (no_connect (at 358.14 185.42))
   (no_connect (at 358.14 50.8))
   (no_connect (at 358.14 175.26))
-  (no_connect (at 358.14 109.22))
   (no_connect (at 358.14 63.5))
   (no_connect (at 358.14 99.06))
-  (no_connect (at 358.14 53.34))
   (no_connect (at 358.14 43.18))
   (no_connect (at 358.14 170.18))
@@
     (stroke (width 0) (type default))
   )
+  (wire (pts (xy 353.06 109.22) (xy 358.14 109.22))
+    (stroke (width 0) (type default))
+  )
   (wire (pts (xy 147.32 181.61) (xy 185.42 181.61))
     (stroke (width 0) (type default))
@@
     (stroke (width 0) (type default))
   )
+  (wire (pts (xy 353.06 165.1) (xy 358.14 165.1))
+    (stroke (width 0) (type default))
+  )
   (wire (pts (xy 347.98 233.68) (xy 347.98 237.49))
     (stroke (width 0) (type default))
@@
     (stroke (width 0) (type default))
   )
+  (wire (pts (xy 353.06 106.68) (xy 353.06 109.22))
+    (stroke (width 0) (type default))
+  )
   (wire (pts (xy 252.73 85.09) (xy 252.73 120.65))
     (stroke (width 0) (type default))
@@
     (stroke (width 0) (type default))
   )
+  (wire (pts (xy 353.06 167.64) (xy 358.14 167.64))
+    (stroke (width 0) (type default))
+  )
   (wire (pts (xy 330.2 245.11) (xy 330.2 247.65))
     (stroke (width 0) (type default))
@@
     (stroke (width 0) (type default))
   )
+  (wire (pts (xy 353.06 170.18) (xy 353.06 167.64))
+    (stroke (width 0) (type default))
+  )
   (wire (pts (xy 340.36 158.75) (xy 340.36 149.86))
     (stroke (width 0) (type default))
   )
+  (wire (pts (xy 353.06 162.56) (xy 353.06 165.1))
+    (stroke (width 0) (type default))
+  )
+  (wire (pts (xy 353.06 55.88) (xy 358.14 55.88))
+    (stroke (width 0) (type default))
+  )
   (wire (pts (xy 347.98 35.56) (xy 358.14 35.56))
     (stroke (width 0) (type default))
@@
     (stroke (width 0) (type solid))
   )
+  (wire (pts (xy 353.06 50.8) (xy 353.06 53.34))
+    (stroke (width 0) (type default))
+  )
   (wire (pts (xy 185.42 143.51) (xy 179.07 143.51))
     (stroke (width 0) (type default))
@@
     (stroke (width 0) (type solid))
   )
+  (wire (pts (xy 353.06 58.42) (xy 353.06 55.88))
+    (stroke (width 0) (type default))
+  )
   (wire (pts (xy 370.84 228.6) (xy 373.38 228.6))
     (stroke (width 0) (type default))
@@
     (stroke (width 0) (type default))
   )
+  (wire (pts (xy 353.06 53.34) (xy 358.14 53.34))
+    (stroke (width 0) (type default))
+  )
   (wire (pts (xy 373.38 208.28) (xy 373.38 213.36))
     (stroke (width 0) (type default))
@@
   )
   (wire (pts (xy 347.98 35.56) (xy 347.98 38.1))
+    (stroke (width 0) (type default))
+  )
+  (wire (pts (xy 353.06 114.3) (xy 353.06 111.76))
+    (stroke (width 0) (type default))
+  )
+  (wire (pts (xy 353.06 111.76) (xy 358.14 111.76))
     (stroke (width 0) (type default))
   )
@@
     )
   )
-  (text "TODO Backplane\nConnector pinout	" (at 336.55 27.94 0)
-    (effects (font (size 3 3) (thickness 0.6) bold (color 255 0 0 1)) (justify left bottom))
-  )
   (text "Raspberry Pi CM4" (at 63.5 31.75 0)
     (effects (font (size 5 5) bold) (justify left bottom))
@@
         (path "/6e8e281e-e30f-459d-852f-231836068db5"
           (reference "U2") (unit 1)
+        )
+      )
+    )
+  )
+  (symbol (lib_id "Power_WUT:0V") (at 353.06 114.3 0) (unit 1)
+    (in_bom no) (on_board no) (dnp no)
+    (property "Reference" "#PWR0306" (at 353.06 114.3 0)
+      (effects (font (size 1.27 1.27)) hide)
+    )
+    (property "Value" "0V" (at 353.06 116.84 0) (do_not_autoplace)
+      (effects (font (size 1.27 1.27)))
+    )
+    (property "Footprint" "" (at 353.06 114.3 0)
+      (effects (font (size 1.27 1.27)) hide)
+    )
+    (property "Datasheet" "" (at 353.06 114.3 0)
+      (effects (font (size 1.27 1.27)) hide)
+    )
+    (pin "1")
+    (instances
+      (project "Master Timing Card"
+        (path "/6e8e281e-e30f-459d-852f-231836068db5"
+          (reference "#PWR0306") (unit 1)
         )
       )
@@
     )
   )
+  (symbol (lib_id "Power_WUT:12V") (at 353.06 162.56 0) (unit 1)
+    (in_bom no) (on_board no) (dnp no) (fields_autoplaced)
+    (property "Reference" "#PWR0304" (at 352.425 165.735 0)
+      (effects (font (size 1.27 1.27)) hide)
+    )
+    (property "Value" "12V" (at 353.06 158.75 0) (do_not_autoplace)
+      (effects (font (size 1.27 1.27)))
+    )
+    (property "Footprint" "" (at 353.06 162.56 0)
+      (effects (font (size 1.27 1.27)) hide)
+    )
+    (property "Datasheet" "" (at 353.06 162.56 0)
+      (effects (font (size 1.27 1.27)) hide)
+    )
+    (pin "1")
+    (instances
+      (project "Master Timing Card"
+        (path "/6e8e281e-e30f-459d-852f-231836068db5"
+          (reference "#PWR0304") (unit 1)
+        )
+      )
+    )
+  )
   (symbol (lib_id "Connector_WUT: Amphenol 86093488613755E1LF") (at 363.22 91.44 0) (unit 2)
     (in_bom yes) (on_board yes) (dnp no) (fields_autoplaced)
@@
     )
   )
+  (symbol (lib_id "Power_WUT:12V") (at 353.06 50.8 0) (unit 1)
+    (in_bom no) (on_board no) (dnp no) (fields_autoplaced)
+    (property "Reference" "#PWR0303" (at 352.425 53.975 0)
+      (effects (font (size 1.27 1.27)) hide)
+    )
+    (property "Value" "12V" (at 353.06 46.99 0) (do_not_autoplace)
+      (effects (font (size 1.27 1.27)))
+    )
+    (property "Footprint" "" (at 353.06 50.8 0)
+      (effects (font (size 1.27 1.27)) hide)
+    )
+    (property "Datasheet" "" (at 353.06 50.8 0)
+      (effects (font (size 1.27 1.27)) hide)
+    )
+    (pin "1")
+    (instances
+      (project "Master Timing Card"
+        (path "/6e8e281e-e30f-459d-852f-231836068db5"
+          (reference "#PWR0303") (unit 1)
+        )
+      )
+    )
+  )
   (symbol (lib_id "AAA_Preferred_WUT:Littelfuse AQ3522-01LTG") (at 285.75 241.3 90) (unit 1)
     (in_bom yes) (on_board yes) (dnp no) (fields_autoplaced)
@@
         (path "/6e8e281e-e30f-459d-852f-231836068db5"
           (reference "#PWR014") (unit 1)
+        )
+      )
+    )
+  )
+  (symbol (lib_id "Power_WUT:0V") (at 353.06 58.42 0) (unit 1)
+    (in_bom no) (on_board no) (dnp no)
+    (property "Reference" "#PWR0307" (at 353.06 58.42 0)
+      (effects (font (size 1.27 1.27)) hide)
+    )
+    (property "Value" "0V" (at 353.06 60.96 0) (do_not_autoplace)
+      (effects (font (size 1.27 1.27)))
+    )
+    (property "Footprint" "" (at 353.06 58.42 0)
+      (effects (font (size 1.27 1.27)) hide)
+    )
+    (property "Datasheet" "" (at 353.06 58.42 0)
+      (effects (font (size 1.27 1.27)) hide)
+    )
+    (pin "1")
+    (instances
+      (project "Master Timing Card"
+        (path "/6e8e281e-e30f-459d-852f-231836068db5"
+          (reference "#PWR0307") (unit 1)
         )
       )
@@
         (path "/6e8e281e-e30f-459d-852f-231836068db5"
           (reference "#PWR05") (unit 1)
+        )
+      )
+    )
+  )
+  (symbol (lib_id "Power_WUT:0V") (at 353.06 170.18 0) (unit 1)
+    (in_bom no) (on_board no) (dnp no)
+    (property "Reference" "#PWR0305" (at 353.06 170.18 0)
+      (effects (font (size 1.27 1.27)) hide)
+    )
+    (property "Value" "0V" (at 353.06 172.72 0) (do_not_autoplace)
+      (effects (font (size 1.27 1.27)))
+    )
+    (property "Footprint" "" (at 353.06 170.18 0)
+      (effects (font (size 1.27 1.27)) hide)
+    )
+    (property "Datasheet" "" (at 353.06 170.18 0)
+      (effects (font (size 1.27 1.27)) hide)
+    )
+    (pin "1")
+    (instances
+      (project "Master Timing Card"
+        (path "/6e8e281e-e30f-459d-852f-231836068db5"
+          (reference "#PWR0305") (unit 1)
         )
       )
@@
         )
       )
+    )
+  )
+  (symbol (lib_id "Power_WUT:12V") (at 353.06 106.68 0) (unit 1)
+    (in_bom no) (on_board no) (dnp no) (fields_autoplaced)
+    (property "Reference" "#PWR0302" (at 352.425 109.855 0)
+      (effects (font (size 1.27 1.27)) hide)
+    )
+    (property "Value" "12V" (at 353.06 102.87 0) (do_not_autoplace)
+      (effects (font (size 1.27 1.27)))
+    )
+    (property "Footprint" "" (at 353.06 106.68 0)
+      (effects (font (size 1.27 1.27)) hide)
+    )
+    (property "Datasheet" "" (at 353.06 106.68 0)
+      (effects (font (size 1.27 1.27)) hide)
+    )
+    (pin "1")
+    (instances
+      (project "Master Timing Card"
+        (path "/6e8e281e-e30f-459d-852f-231836068db5"
+          (reference "#PWR0302") (unit 1)
+        )
+      )
