File: Master Timing Card.kicad_sch (KiCad schematic)
At the start: 28 parts, among them CN1 Samtec GRF1-J-P-08-E-RA-TH1, CN2 Amphenol 86093488613755E1LF, U1 Analog MAX3483ESA+, U2 DS2431P+

Commit message: .
Parts:
- LAYOUT1, LAYOUT2, LAYOUT3: now left out of the parts list
Changed lines of the file:
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@@
 		(unit 1)
 		(exclude_from_sim no)
-		(in_bom yes)
+		(in_bom no)
 		(on_board yes)
 		(dnp no)
@@
 		(unit 1)
 		(exclude_from_sim no)
-		(in_bom yes)
+		(in_bom no)
 		(on_board yes)
 		(dnp no)
@@
 		(unit 1)
 		(exclude_from_sim no)
-		(in_bom yes)
+		(in_bom no)
 		(on_board yes)
 		(dnp no)
