File: cm4_io.kicad_sch (KiCad schematic)
At the start: 20 parts, among them CN7 104031-0811, J1 Connector_RJ45_Magjack_Abraco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, Q4 onsemi FDC6330L

Commit message: Added M.2 SSD
Parts:
- CN4: MPN DF40C-100DS-0.4V -> DF40C-100DS-0.4V(51)
Changed lines of the file:
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@@
     )
   )
-  (symbol (lib_name "ComputeModule4-GPIO_2") (lib_id "Modules_WUT:ComputeModule4-GPIO") (at 106.68 46.99 0) (unit 2)
+  (symbol (lib_id "Modules_WUT:ComputeModule4-GPIO") (at 106.68 46.99 0) (unit 2)
     (in_bom yes) (on_board yes) (dnp no) (fields_autoplaced)
     (property "Reference" "CN4" (at 106.68 41.91 0)
@@
       (effects (font (size 1.27 1.27)) hide)
     )
-    (property "MPN" "DF40C-100DS-0.4V" (at 106.68 46.99 0)
+    (property "MPN" "DF40C-100DS-0.4V(51)" (at 106.68 46.99 0)
       (effects (font (size 1.27 1.27)) hide)
     )

Commit message: Added ESD and tided up PSU
Parts:
- added D5, D6: TPD4E05U06DQA, Diode_WUT:TPD4E05U06DQA, symbol Diode_WUT:TI_TPD4E05U06
Connections:
- net 0V: now also D5.3, D5.8, D6.3, D6.8
- net at CN4.10 (Ethernet_Pair0_N), J1.2: now also D5.2, D5.9 (NC)
- net at CN4.11 (Ethernet_Pair2_P), J1.7: now also D6.1, D6.10 (NC)
- net at CN4.12 (Ethernet_Pair0_P), J1.1: now also D5.1, D5.10 (NC)
- net at CN4.3 (Ethernet_Pair3_P), J1.9: now also D6.4, D6.7 (NC)
- net at CN4.4 (Ethernet_Pair1_P), J1.3: now also D5.4, D5.7 (NC)
- net at CN4.5 (Ethernet_Pair3_N), J1.10: now also D6.5, D6.6 (NC)
- net at CN4.6 (Ethernet_Pair1_N), J1.4: now also D5.5, D5.6 (NC)
- net at CN4.9 (Ethernet_Pair2_N), J1.8: now also D6.2, D6.9 (NC)
- no-connect marks 3 -> 4
Other:
- moved on the sheet: C116, C117, C70, CN7, D1, D2, J1, Q4, R38, R39, R49, R50

Commit message: started on power
Parts:
- CN7: footprint Connector_Card:microSD_HC_Molex_104031-0811 -> Connector_WUT:microSD_HC_Molex_104031-0811
Connections:
- no-connect marks 4 -> 8
Changed lines of the file:
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@@
   )
   (no_connect (at 83.82 46.99))
+  (no_connect (at 83.82 74.93))
   (no_connect (at 129.54 77.47))
+  (no_connect (at 83.82 69.85))
   (no_connect (at 193.04 160.02))
   (no_connect (at 129.54 90.17))
+  (no_connect (at 83.82 72.39))
+  (no_connect (at 83.82 67.31))
   (wire (pts (xy 158.75 46.99) (xy 226.06 46.99))
     (stroke (width 0) (type default))
@@
       (effects (font (size 1.27 1.27)))
     )
-    (property "Footprint" "Connector_Card:microSD_HC_Molex_104031-0811" (at 257.81 179.07 0)
-      (effects (font (size 1.27 1.27)) hide)
-    )
+    (property "Footprint" "Connector_WUT:microSD_HC_Molex_104031-0811" (at 257.81 179.07 0)
+      (effects (font (size 1.27 1.27)) hide)
+    )

Commit message: schematic complete
Connections:
- net 0V: now also CN7.10 (DET_A)
- no-connect marks 8 -> 9
Changed lines of the file:
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@@
   (junction (at 173.99 57.15) (diameter 0) (color 0 0 0 0)
   )
+  (junction (at 119.38 168.91) (diameter 0) (color 0 0 0 0)
+  )
   (junction (at 158.75 46.99) (diameter 0) (color 0 0 0 0)
   )
@@
   (junction (at 158.75 88.9) (diameter 0) (color 0 0 0 0)
   )
+  (junction (at 231.14 190.5) (diameter 0) (color 0 0 0 0)
+  )
   (junction (at 191.77 62.23) (diameter 0) (color 0 0 0 0)
   )
@@
   )
   (no_connect (at 83.82 46.99))
+  (no_connect (at 267.97 82.55))
   (no_connect (at 83.82 74.93))
   (no_connect (at 129.54 77.47))
@@
     (stroke (width 0) (type default))
   )
+  (wire (pts (xy 231.14 190.5) (xy 231.14 182.88))
+    (stroke (width 0) (type default))
+  )
   (wire (pts (xy 109.22 171.45) (xy 113.03 171.45))
     (stroke (width 0) (type default))
@@
     (stroke (width 0) (type default))
   )
-  (wire (pts (xy 231.14 193.04) (xy 231.14 182.88))
+  (wire (pts (xy 231.14 193.04) (xy 231.14 190.5))
     (stroke (width 0) (type default))
   )
@@
     (stroke (width 0) (type default))
   )
-  (wire (pts (xy 113.03 168.91) (xy 124.46 168.91))
+  (wire (pts (xy 113.03 168.91) (xy 119.38 168.91))
     (stroke (width 0) (type default))
   )
@@
     (stroke (width 0) (type default))
   )
+  (wire (pts (xy 231.14 190.5) (xy 233.68 190.5))
+    (stroke (width 0) (type default))
+  )
   (wire (pts (xy 189.23 88.9) (xy 189.23 91.44))
     (stroke (width 0) (type default))
@@
   )
   (wire (pts (xy 257.81 90.17) (xy 267.97 90.17))
+    (stroke (width 0) (type default))
+  )
+  (wire (pts (xy 119.38 168.91) (xy 124.46 168.91))
     (stroke (width 0) (type default))
   )
@@
         )
       )
+    )
+  )
+  (symbol (lib_id "Power_WUT:PWR_FLAG") (at 119.38 168.91 0) (unit 1)
+    (in_bom yes) (on_board yes) (dnp no) (fields_autoplaced)
+    (property "Reference" "#FLG032" (at 119.38 167.005 0)
+      (effects (font (size 1.27 1.27)) hide)
+    )
+    (property "Value" "PWR_FLAG" (at 119.38 165.1 0)
+      (effects (font (size 1.27 1.27)) hide)
+    )
+    (property "Footprint" "" (at 119.38 168.91 0)
+      (effects (font (size 1.27 1.27)) hide)
+    )
+    (property "Datasheet" "~" (at 119.38 168.91 0)
+      (effects (font (size 1.27 1.27)) hide)
+    )
+    (pin "1")
+    (instances
+      (project "Master Timing Card"
+        (path "/6e8e281e-e30f-459d-852f-231836068db5/c1c9a6e7-67cd-4895-bef3-80d2d409d5a5"
+          (reference "#FLG032") (unit 1)
+        )
+      )

Commit message: Moved to preferred library
Parts:
- C116, C117, C70: symbol Auto_Library_WUT:Yageo CC0402KRX7R8BB104 -> Preferred_WUT:Yageo CC0402KRX7R8BB104
- R38, R39: symbol Auto_Library_WUT:KOA Speer RK73H1ETTP1001F -> Preferred_WUT:KOA Speer RK73H1ETTP1001F
- R49, R50: symbol Auto_Library_WUT:KOA Speer RK73H1ETTP1002F -> Preferred_WUT:KOA Speer RK73H1ETTP1002F
- R51: symbol Auto_Library_WUT:KOA Speer RK73H1ETTP1000F -> Preferred_WUT:KOA Speer RK73H1ETTP1000F
- R7: symbol Auto_Library_WUT:KOA Speer RK73H1ETTP33R0F -> Preferred_WUT:KOA Speer RK73H1ETTP33R0F
Connections:
- net ETHA_P: now reaches CN4.12 (Ethernet_Pair0_P), D5.1, D5.10 (NC), J1.1
- net ETHA_N: now reaches CN4.10 (Ethernet_Pair0_N), D5.2, D5.9 (NC), J1.2
- net ETHB_P: now reaches CN4.4 (Ethernet_Pair1_P), D5.4, D5.7 (NC), J1.3
- net ETHB_N: now reaches CN4.6 (Ethernet_Pair1_N), D5.5, D5.6 (NC), J1.4
- net ETHC_P: now reaches CN4.11 (Ethernet_Pair2_P), D6.1, D6.10 (NC), J1.7
- net ETHD_P: now reaches CN4.3 (Ethernet_Pair3_P), D6.4, D6.7 (NC), J1.9
- net ETHD_N: now reaches CN4.5 (Ethernet_Pair3_N), D6.5, D6.6 (NC), J1.10
- net ETHC_N: now reaches CN4.9 (Ethernet_Pair2_N), D6.2, D6.9 (NC), J1.8
Changed lines of the file:
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@@
     (effects (font (size 1.27 1.27)) (justify right bottom))
   )
+  (label "ETHB_P" (at 132.08 54.61 0) (fields_autoplaced)
+    (effects (font (size 1.27 1.27)) (justify left bottom))
+  )
   (label "SD_DAT2" (at 157.48 170.18 0) (fields_autoplaced)
     (effects (font (size 1.27 1.27)) (justify left bottom))
   )
+  (label "ETHA_P" (at 132.08 46.99 0) (fields_autoplaced)
+    (effects (font (size 1.27 1.27)) (justify left bottom))
+  )
   (label "SD_DAT3" (at 157.48 172.72 0) (fields_autoplaced)
     (effects (font (size 1.27 1.27)) (justify left bottom))
@@
   )
   (label "SD_DAT3" (at 46.99 64.77 0) (fields_autoplaced)
+    (effects (font (size 1.27 1.27)) (justify left bottom))
+  )
+  (label "ETHA_N" (at 132.08 49.53 0) (fields_autoplaced)
     (effects (font (size 1.27 1.27)) (justify left bottom))
   )
@@
     (effects (font (size 1.27 1.27)) (justify left bottom))
   )
+  (label "ETHB_N" (at 132.08 57.15 0) (fields_autoplaced)
+    (effects (font (size 1.27 1.27)) (justify left bottom))
+  )
+  (label "ETHD_P" (at 132.08 69.85 0) (fields_autoplaced)
+    (effects (font (size 1.27 1.27)) (justify left bottom))
+  )
   (label "~{ETH_LINK}" (at 142.24 80.01 180) (fields_autoplaced)
     (effects (font (size 1.27 1.27)) (justify right bottom))
@@
     (effects (font (size 1.27 1.27)) (justify left bottom))
   )
+  (label "ETHC_P" (at 132.08 62.23 0) (fields_autoplaced)
+    (effects (font (size 1.27 1.27)) (justify left bottom))
+  )
+  (label "ETHC_N" (at 132.08 64.77 0) (fields_autoplaced)
+    (effects (font (size 1.27 1.27)) (justify left bottom))
+  )
   (label "SD_PWR_ON" (at 68.58 181.61 0) (fields_autoplaced)
     (effects (font (size 1.27 1.27)) (justify left bottom))
@@
   )
   (label "~{ETH_ACT}" (at 257.81 90.17 0) (fields_autoplaced)
+    (effects (font (size 1.27 1.27)) (justify left bottom))
+  )
+  (label "ETHD_N" (at 132.08 72.39 0) (fields_autoplaced)
     (effects (font (size 1.27 1.27)) (justify left bottom))
   )
@@
     )
   )
-  (symbol (lib_id "Auto_Library_WUT:Yageo CC0402KRX7R8BB104") (at 113.03 179.07 0) (unit 1)
+  (symbol (lib_id "Preferred_WUT:Yageo CC0402KRX7R8BB104") (at 113.03 179.07 0) (unit 1)
     (in_bom yes) (on_board yes) (dnp yes) (fields_autoplaced)
     (property "Reference" "C117" (at 115.57 176.53 0) (do_not_autoplace)
@@
     )
   )
-  (symbol (lib_id "Auto_Library_WUT:KOA Speer RK73H1ETTP1001F") (at 254 93.98 90) (unit 1)
+  (symbol (lib_id "Preferred_WUT:KOA Speer RK73H1ETTP1001F") (at 254 93.98 90) (unit 1)
     (in_bom yes) (on_board yes) (dnp no)
     (property "Reference" "R38" (at 254 91.44 90)
@@
     )
   )
-  (symbol (lib_id "Auto_Library_WUT:KOA Speer RK73H1ETTP33R0F") (at 72.39 64.77 270) (mirror x) (unit 1)
+  (symbol (lib_id "Preferred_WUT:KOA Speer RK73H1ETTP33R0F") (at 72.39 64.77 270) (mirror x) (unit 1)
     (in_bom yes) (on_board yes) (dnp yes)
     (property "Reference" "R7" (at 66.04 63.5 90)
@@
     )
   )
-  (symbol (lib_id "Auto_Library_WUT:KOA Speer RK73H1ETTP33R0F") (at 72.39 85.09 270) (mirror x) (unit 1)
+  (symbol (lib_id "Preferred_WUT:KOA Speer RK73H1ETTP33R0F") (at 72.39 85.09 270) (mirror x) (unit 1)
     (in_bom yes) (on_board yes) (dnp yes)
     (property "Reference" "R7" (at 66.04 83.82 90)
@@
     )
   )
-  (symbol (lib_id "Auto_Library_WUT:KOA Speer RK73H1ETTP33R0F") (at 72.39 59.69 270) (mirror x) (unit 1)
+  (symbol (lib_id "Preferred_WUT:KOA Speer RK73H1ETTP33R0F") (at 72.39 59.69 270) (mirror x) (unit 1)
     (in_bom yes) (on_board yes) (dnp yes)
     (property "Reference" "R7" (at 66.04 58.42 90)
@@
     )
   )
-  (symbol (lib_id "Auto_Library_WUT:KOA Speer RK73H1ETTP33R0F") (at 72.39 62.23 270) (mirror x) (unit 1)
+  (symbol (lib_id "Preferred_WUT:KOA Speer RK73H1ETTP33R0F") (at 72.39 62.23 270) (mirror x) (unit 1)
     (in_bom yes) (on_board yes) (dnp yes)
     (property "Reference" "R7" (at 66.04 60.96 90)
@@
     )
   )
-  (symbol (lib_id "Auto_Library_WUT:Yageo CC0402KRX7R8BB104") (at 250.19 27.94 0) (unit 1)
+  (symbol (lib_id "Preferred_WUT:Yageo CC0402KRX7R8BB104") (at 250.19 27.94 0) (unit 1)
     (in_bom yes) (on_board yes) (dnp no) (fields_autoplaced)
     (property "Reference" "C70" (at 252.73 25.4 0) (do_not_autoplace)
@@
     )
   )
-  (symbol (lib_id "Auto_Library_WUT:Yageo CC0402KRX7R8BB104") (at 175.26 153.67 0) (unit 1)
+  (symbol (lib_id "Preferred_WUT:Yageo CC0402KRX7R8BB104") (at 175.26 153.67 0) (unit 1)
     (in_bom yes) (on_board yes) (dnp yes) (fields_autoplaced)
     (property "Reference" "C116" (at 177.8 151.13 0) (do_not_autoplace)
@@
     )
   )
-  (symbol (lib_id "Auto_Library_WUT:KOA Speer RK73H1ETTP33R0F") (at 72.39 57.15 270) (mirror x) (unit 1)
+  (symbol (lib_id "Preferred_WUT:KOA Speer RK73H1ETTP33R0F") (at 72.39 57.15 270) (mirror x) (unit 1)
     (in_bom yes) (on_board yes) (dnp yes)
     (property "Reference" "R7" (at 66.04 55.88 90)
@@
     )
   )
-  (symbol (lib_id "Auto_Library_WUT:KOA Speer RK73H1ETTP1002F") (at 81.28 186.69 0) (unit 1)
+  (symbol (lib_id "Preferred_WUT:KOA Speer RK73H1ETTP1002F") (at 81.28 186.69 0) (unit 1)
     (in_bom yes) (on_board yes) (dnp yes) (fields_autoplaced)
     (property "Reference" "R50" (at 83.82 185.42 0)
@@
     )
   )
-  (symbol (lib_id "Auto_Library_WUT:KOA Speer RK73H1ETTP33R0F") (at 72.39 80.01 270) (mirror x) (unit 1)
+  (symbol (lib_id "Preferred_WUT:KOA Speer RK73H1ETTP33R0F") (at 72.39 80.01 270) (mirror x) (unit 1)
     (in_bom yes) (on_board yes) (dnp yes)
     (property "Reference" "R7" (at 66.04 78.74 90)
@@
     )
   )
-  (symbol (lib_id "Auto_Library_WUT:KOA Speer RK73H1ETTP1002F") (at 81.28 173.99 0) (unit 1)
+  (symbol (lib_id "Preferred_WUT:KOA Speer RK73H1ETTP1002F") (at 81.28 173.99 0) (unit 1)
     (in_bom yes) (on_board yes) (dnp yes) (fields_autoplaced)
     (property "Reference" "R49" (at 83.82 172.72 0)
@@
     )
   )
-  (symbol (lib_id "Auto_Library_WUT:KOA Speer RK73H1ETTP1000F") (at 72.39 52.07 90) (unit 1)
+  (symbol (lib_id "Preferred_WUT:KOA Speer RK73H1ETTP1000F") (at 72.39 52.07 90) (unit 1)
     (in_bom yes) (on_board yes) (dnp yes) (fields_autoplaced)
     (property "Reference" "R51" (at 72.39 45.72 90)
@@
     )
   )
-  (symbol (lib_id "Auto_Library_WUT:KOA Speer RK73H1ETTP1001F") (at 254 86.36 90) (unit 1)
+  (symbol (lib_id "Preferred_WUT:KOA Speer RK73H1ETTP1001F") (at 254 86.36 90) (unit 1)
     (in_bom yes) (on_board yes) (dnp no)
     (property "Reference" "R39" (at 254 83.82 90)

Commit message: layout progress
Parts:
- removed C70: 100n, Capacitor_SMD:C_0402_1005Metric, symbol Preferred_WUT:Yageo CC0402KRX7R8BB104
- C100: renamed from C117; symbol Preferred_WUT:Yageo CC0402KRX7R8BB104 -> AAA_Preferred_WUT:Yageo CC0402KRX7R8BB104
- C101: renamed from C116; symbol Preferred_WUT:Yageo CC0402KRX7R8BB104 -> AAA_Preferred_WUT:Yageo CC0402KRX7R8BB104
- CN14: renamed from J1; value Connector_RJ45_Magjack_Abracon_ARJM11D7-502-AB-EW2 -> 1-2301994-2; footprint Connector_WUT:Connector_RJ45_Magjack_Abracon_ARJM11D7-502-AB-EW2 -> Connector_WUT:TE_1-2301994-2; symbol Connector_WUT:Connector_RJ45_Magjack_Abracon_ARJM11D7-502-AB-EW2 -> Connector_WUT:RJ45_Magjack_TE_1-2301994-2; MPN ARJM11D7-502-AB-EW2 -> 1-2301994-2; Manufacturer (none) -> TE Connectivity
- R87: renamed from R51; symbol Preferred_WUT:KOA Speer RK73H1ETTP1000F -> AAA_Preferred_WUT:KOA Speer RK73H1ETTP1000F
- R88, R89, R90, R91, R92, R93: renamed from R7; symbol Preferred_WUT:KOA Speer RK73H1ETTP33R0F -> AAA_Preferred_WUT:KOA Speer RK73H1ETTP33R0F
- R94: renamed from R49; symbol Preferred_WUT:KOA Speer RK73H1ETTP1002F -> AAA_Preferred_WUT:KOA Speer RK73H1ETTP1002F
- R95: renamed from R50; symbol Preferred_WUT:KOA Speer RK73H1ETTP1002F -> AAA_Preferred_WUT:KOA Speer RK73H1ETTP1002F
- R96: renamed from R39; symbol Preferred_WUT:KOA Speer RK73H1ETTP1001F -> AAA_Preferred_WUT:KOA Speer RK73H1ETTP1001F
- R97: renamed from R38; symbol Preferred_WUT:KOA Speer RK73H1ETTP1001F -> AAA_Preferred_WUT:KOA Speer RK73H1ETTP1001F
- renumbered CN7 to CN13, D2 to D20, D5 to D21, D1 to D22, D6 to D23, Q4 to Q5
Connections:
- net 0V: now also CN14.10
- net ETHA_N: now also CN14.3, D23.4, D23.7 (NC); no longer CN14.2, D21.2, D21.9 (NC)
- net ETHA_P: now also CN14.2, D23.5, D23.6 (NC); no longer CN14.1, D21.1, D21.10 (NC)
- net ETHB_N: now also CN14.5, D23.1, D23.10 (NC); no longer CN14.4, D21.5, D21.6 (NC)
- net ETHB_P: now also CN14.4, D23.2, D23.9 (NC); no longer CN14.3, D21.4, D21.7 (NC)
- net ETHC_N: now also CN14.7, D21.4, D21.7 (NC); no longer CN14.8, D23.2, D23.9 (NC)
- net ETHC_P: now also CN14.6, D21.5, D21.6 (NC); no longer CN14.7, D23.1, D23.10 (NC)
- net ETHD_N: now also CN14.9, D21.1, D21.10 (NC); no longer CN14.10, D23.5, D23.6 (NC)
- net ETHD_P: now also CN14.8, D21.2, D21.9 (NC); no longer CN14.9, D23.4, D23.7 (NC)

Commit message: getting there
Parts:
- removed C100, C101: 100n, Capacitor_SMD:C_0402_1005Metric, symbol AAA_Preferred_WUT:Yageo CC0402KRX7R8BB104
- removed CN13: 104031-0811, Connector_WUT:microSD_HC_Molex_104031-0811, symbol Connector_WUT:Molex_104031-0811
- removed D20: 5V0, Diode_SMD:D_SOD-323, symbol Auto_Library_WUT:nexperia PESD5V0U1UA,115
- removed D22: ECLAMP2410P, Diode_WUT:Semtech_ECLAMP2410P, symbol Diode_WUT:Semtech_EClamp2410P
- removed Q5: onsemi FDC6330L, Package_TO_SOT_SMD:TSOT-23-6, symbol Transistor_WUT:onsemi_FDC6330L
- removed R87: 100R, Resistor_SMD:R_0402_1005Metric, symbol AAA_Preferred_WUT:KOA Speer RK73H1ETTP1000F
- removed R88, R89, R90, R91, R92, R93: 33R, Resistor_SMD:R_0402_1005Metric, symbol AAA_Preferred_WUT:KOA Speer RK73H1ETTP33R0F
- removed R94, R95: 10k, Resistor_SMD:R_0402_1005Metric, symbol AAA_Preferred_WUT:KOA Speer RK73H1ETTP1002F
Connections:
- no-connect marks 9 -> 15
Other:
- note removed: "Recommend to not use Lite versions for reliability but footprints are provided in case"
