File: cm4_io.kicad_sch (KiCad schematic)
At the start: 6 parts, among them CN14 1-2301994-2

Commit message: committing before attempting scripting
Parts:
- renumbered CN14 to CN13, D21 to D20, D23 to D21, R96 to R89, R97 to R90
Connections:
- net SH: now reaches CN13.11 (SHIELD)
Changed lines of the file:
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@@
   (no_connect (at 83.82 57.15))
   (no_connect (at 83.82 46.99))
-  (no_connect (at 267.97 82.55))
+  (no_connect (at 264.16 82.55))
   (no_connect (at 83.82 74.93))
   (no_connect (at 83.82 85.09))
@@
     (stroke (width 0) (type default))
   )
+  (wire (pts (xy 260.35 80.01) (xy 260.35 78.74))
+    (stroke (width 0) (type default))
+  )
   (wire (pts (xy 226.06 48.26) (xy 226.06 49.53))
     (stroke (width 0) (type default))
@@
     (stroke (width 0) (type default))
   )
+  (wire (pts (xy 260.35 78.74) (xy 267.97 78.74))
+    (stroke (width 0) (type default))
+  )
   (wire (pts (xy 158.75 72.39) (xy 226.06 72.39))
     (stroke (width 0) (type default))
@@
     (stroke (width 0) (type default))
   )
-  (wire (pts (xy 262.89 78.74) (xy 267.97 78.74))
-    (stroke (width 0) (type default))
-  )
   (wire (pts (xy 257.81 86.36) (xy 267.97 86.36))
     (stroke (width 0) (type default))
@@
     (stroke (width 0) (type default))
   )
-  (wire (pts (xy 262.89 81.28) (xy 262.89 78.74))
-    (stroke (width 0) (type default))
-  )
   (wire (pts (xy 171.45 88.9) (xy 173.99 88.9))
     (stroke (width 0) (type default))
@@
   )
   (wire (pts (xy 196.85 54.61) (xy 226.06 54.61))
+    (stroke (width 0) (type default))
+  )
+  (wire (pts (xy 264.16 82.55) (xy 267.97 82.55))
     (stroke (width 0) (type default))
   )
@@
     (effects (font (size 1.27 1.27)) (justify left bottom))
   )
+  (label "SH" (at 265.43 82.55 0) (fields_autoplaced)
+    (effects (font (size 1.27 1.27)) (justify left bottom))
+  )
   (label "~{ETH_ACT}" (at 257.81 90.17 0) (fields_autoplaced)
     (effects (font (size 1.27 1.27)) (justify left bottom))
@@
   (symbol (lib_id "Power_WUT:0V") (at 201.93 116.84 0) (unit 1)
     (in_bom no) (on_board no) (dnp no) (fields_autoplaced)
-    (property "Reference" "#PWR0218" (at 201.93 116.84 0)
+    (property "Reference" "#PWR0212" (at 201.93 116.84 0)
       (effects (font (size 1.27 1.27)) hide)
     )
@@
       (project "Master Timing Card"
         (path "/6e8e281e-e30f-459d-852f-231836068db5/c1c9a6e7-67cd-4895-bef3-80d2d409d5a5"
-          (reference "#PWR0218") (unit 1)
+          (reference "#PWR0212") (unit 1)
         )
       )
@@
   (symbol (lib_id "Power_WUT:0V") (at 158.75 116.84 0) (unit 1)
     (in_bom no) (on_board no) (dnp no) (fields_autoplaced)
-    (property "Reference" "#PWR0212" (at 158.75 116.84 0)
+    (property "Reference" "#PWR0209" (at 158.75 116.84 0)
       (effects (font (size 1.27 1.27)) hide)
     )
@@
       (project "Master Timing Card"
         (path "/6e8e281e-e30f-459d-852f-231836068db5/c1c9a6e7-67cd-4895-bef3-80d2d409d5a5"
-          (reference "#PWR0212") (unit 1)
+          (reference "#PWR0209") (unit 1)
         )
       )
@@
   (symbol (lib_id "Power_WUT:0V") (at 191.77 116.84 0) (unit 1)
     (in_bom no) (on_board no) (dnp no) (fields_autoplaced)
-    (property "Reference" "#PWR0216" (at 191.77 116.84 0)
+    (property "Reference" "#PWR0211" (at 191.77 116.84 0)
       (effects (font (size 1.27 1.27)) hide)
     )
@@
       (project "Master Timing Card"
         (path "/6e8e281e-e30f-459d-852f-231836068db5/c1c9a6e7-67cd-4895-bef3-80d2d409d5a5"
-          (reference "#PWR0216") (unit 1)
+          (reference "#PWR0211") (unit 1)
         )
       )
@@
   (symbol (lib_id "AAA_Preferred_WUT:KOA Speer RK73H1ETTP1001F") (at 254 93.98 90) (unit 1)
     (in_bom yes) (on_board yes) (dnp no)
-    (property "Reference" "R97" (at 254 91.44 90)
+    (property "Reference" "R90" (at 254 91.44 90)
       (effects (font (size 1.27 1.27)))
     )
@@
       (project "Master Timing Card"
         (path "/6e8e281e-e30f-459d-852f-231836068db5/c1c9a6e7-67cd-4895-bef3-80d2d409d5a5"
-          (reference "R97") (unit 1)
+          (reference "R90") (unit 1)
         )
       )
@@
   (symbol (lib_id "Power_WUT:0V") (at 168.91 116.84 0) (unit 1)
     (in_bom no) (on_board no) (dnp no) (fields_autoplaced)
-    (property "Reference" "#PWR0213" (at 168.91 116.84 0)
+    (property "Reference" "#PWR0210" (at 168.91 116.84 0)
       (effects (font (size 1.27 1.27)) hide)
     )
@@
       (project "Master Timing Card"
         (path "/6e8e281e-e30f-459d-852f-231836068db5/c1c9a6e7-67cd-4895-bef3-80d2d409d5a5"
-          (reference "#PWR0213") (unit 1)
+          (reference "#PWR0210") (unit 1)
         )
       )
@@
   (symbol (lib_id "Power_WUT:3V3") (at 247.65 92.71 0) (unit 1)
     (in_bom no) (on_board no) (dnp no)
-    (property "Reference" "#PWR0221" (at 247.015 95.885 0)
+    (property "Reference" "#PWR0214" (at 247.015 95.885 0)
       (effects (font (size 1.27 1.27)) hide)
     )
@@
       (project "Master Timing Card"
         (path "/6e8e281e-e30f-459d-852f-231836068db5/c1c9a6e7-67cd-4895-bef3-80d2d409d5a5"
-          (reference "#PWR0221") (unit 1)
+          (reference "#PWR0214") (unit 1)
         )
       )
@@
   (symbol (lib_id "Diode_WUT:TI_TPD4E05U06") (at 163.83 104.14 0) (unit 1)
     (in_bom yes) (on_board yes) (dnp no)
-    (property "Reference" "D21" (at 170.18 113.03 0) (do_not_autoplace)
+    (property "Reference" "D20" (at 170.18 113.03 0) (do_not_autoplace)
       (effects (font (size 1.27 1.27)) (justify left))
     )
@@
       (project "Master Timing Card"
         (path "/6e8e281e-e30f-459d-852f-231836068db5/c1c9a6e7-67cd-4895-bef3-80d2d409d5a5"
-          (reference "D21") (unit 1)
+          (reference "D20") (unit 1)
         )
       )
@@
   (symbol (lib_id "Power_WUT:3V3") (at 247.65 85.09 0) (unit 1)
     (in_bom no) (on_board no) (dnp no)
-    (property "Reference" "#PWR0220" (at 247.015 88.265 0)
+    (property "Reference" "#PWR0213" (at 247.015 88.265 0)
       (effects (font (size 1.27 1.27)) hide)
     )
@@
       (project "Master Timing Card"
         (path "/6e8e281e-e30f-459d-852f-231836068db5/c1c9a6e7-67cd-4895-bef3-80d2d409d5a5"
-          (reference "#PWR0220") (unit 1)
+          (reference "#PWR0213") (unit 1)
         )
       )
@@
     )
   )
-  (symbol (lib_id "Power_WUT:0V") (at 262.89 81.28 0) (unit 1)
+  (symbol (lib_id "Power_WUT:0V") (at 260.35 80.01 0) (unit 1)
     (in_bom no) (on_board no) (dnp no) (fields_autoplaced)
-    (property "Reference" "#PWR0222" (at 262.89 81.28 0)
-      (effects (font (size 1.27 1.27)) hide)
-    )
-    (property "Value" "0V" (at 262.89 83.82 0) (do_not_autoplace)
-      (effects (font (size 1.27 1.27)))
-    )
-    (property "Footprint" "" (at 262.89 81.28 0)
-      (effects (font (size 1.27 1.27)) hide)
-    )
-    (property "Datasheet" "" (at 262.89 81.28 0)
-      (effects (font (size 1.27 1.27)) hide)
-    )
-    (pin "1")
-    (instances
-      (project "Master Timing Card"
-        (path "/6e8e281e-e30f-459d-852f-231836068db5/c1c9a6e7-67cd-4895-bef3-80d2d409d5a5"
-          (reference "#PWR0222") (unit 1)
+    (property "Reference" "#PWR0215" (at 260.35 80.01 0)
+      (effects (font (size 1.27 1.27)) hide)
+    )
+    (property "Value" "0V" (at 260.35 82.55 0) (do_not_autoplace)
+      (effects (font (size 1.27 1.27)))
+    )
+    (property "Footprint" "" (at 260.35 80.01 0)
+      (effects (font (size 1.27 1.27)) hide)
+    )
+    (property "Datasheet" "" (at 260.35 80.01 0)
+      (effects (font (size 1.27 1.27)) hide)
+    )
+    (pin "1")
+    (instances
+      (project "Master Timing Card"
+        (path "/6e8e281e-e30f-459d-852f-231836068db5/c1c9a6e7-67cd-4895-bef3-80d2d409d5a5"
+          (reference "#PWR0215") (unit 1)
         )
       )
@@
   (symbol (lib_id "Diode_WUT:TI_TPD4E05U06") (at 196.85 104.14 0) (unit 1)
     (in_bom yes) (on_board yes) (dnp no)
-    (property "Reference" "D23" (at 203.2 113.03 0) (do_not_autoplace)
+    (property "Reference" "D21" (at 203.2 113.03 0) (do_not_autoplace)
       (effects (font (size 1.27 1.27)) (justify left))
     )
@@
       (project "Master Timing Card"
         (path "/6e8e281e-e30f-459d-852f-231836068db5/c1c9a6e7-67cd-4895-bef3-80d2d409d5a5"
-          (reference "D23") (unit 1)
+          (reference "D21") (unit 1)
         )
       )
@@
   (symbol (lib_id "Connector_WUT:RJ45_Magjack_TE_1-2301994-2") (at 283.21 55.88 0) (unit 1)
     (in_bom yes) (on_board yes) (dnp no)
-    (property "Reference" "CN14" (at 281.94 39.37 0)
+    (property "Reference" "CN13" (at 281.94 39.37 0)
       (effects (font (size 1.27 1.27)) (justify left))
     )
@@
       (project "Master Timing Card"
         (path "/6e8e281e-e30f-459d-852f-231836068db5/c1c9a6e7-67cd-4895-bef3-80d2d409d5a5"
-          (reference "CN14") (unit 1)
+          (reference "CN13") (unit 1)
         )
       )
@@
   (symbol (lib_id "AAA_Preferred_WUT:KOA Speer RK73H1ETTP1001F") (at 254 86.36 90) (unit 1)
     (in_bom yes) (on_board yes) (dnp no)
-    (property "Reference" "R96" (at 254 83.82 90)
+    (property "Reference" "R89" (at 254 83.82 90)
       (effects (font (size 1.27 1.27)))
     )
@@
       (project "Master Timing Card"
         (path "/6e8e281e-e30f-459d-852f-231836068db5/c1c9a6e7-67cd-4895-bef3-80d2d409d5a5"
-          (reference "R96") (unit 1)
-        )
-      )
+          (reference "R89") (unit 1)
+        )
+      )
