File: rc32504.kicad_sch (KiCad schematic)
At the start: 62 parts, among them T1 TC2-72T+, T2 TC2-72T+, T4 TC2-72T+, T7 TC2-72T+, U13 LT3045IDD#PBF, U4 RC32504A000GNK#BB0

Commit message: layout progress
Parts:
- C57: renamed from C40; symbol Preferred_WUT:Yageo CC0402KRX7R8BB104 -> AAA_Preferred_WUT:Yageo CC0402KRX7R8BB104
- C58: renamed from C41; symbol Preferred_WUT:Yageo CC0402KRX7R8BB104 -> AAA_Preferred_WUT:Yageo CC0402KRX7R8BB104
- C59: renamed from C45; symbol Preferred_WUT:Yageo CC0402KRX7R8BB104 -> AAA_Preferred_WUT:Yageo CC0402KRX7R8BB104
- C60: renamed from C49; symbol Preferred_WUT:Yageo CC0402KRX7R8BB104 -> AAA_Preferred_WUT:Yageo CC0402KRX7R8BB104
- C61: renamed from C53; symbol Preferred_WUT:Yageo CC0402KRX7R8BB104 -> AAA_Preferred_WUT:Yageo CC0402KRX7R8BB104
- C62: renamed from C56; symbol Preferred_WUT:Yageo CC0402KRX7R8BB104 -> AAA_Preferred_WUT:Yageo CC0402KRX7R8BB104
- C63: renamed from C59; symbol Preferred_WUT:Yageo CC0402KRX7R8BB104 -> AAA_Preferred_WUT:Yageo CC0402KRX7R8BB104
- C71: renamed from C38; symbol Preferred_WUT:Yageo CC0402KRX7R8BB104 -> AAA_Preferred_WUT:Yageo CC0402KRX7R8BB104
- C72: renamed from C43; symbol Preferred_WUT:Yageo CC0402KRX7R8BB104 -> AAA_Preferred_WUT:Yageo CC0402KRX7R8BB104
- C73: renamed from C47; symbol Preferred_WUT:Yageo CC0402KRX7R8BB104 -> AAA_Preferred_WUT:Yageo CC0402KRX7R8BB104
- C74: renamed from C51; symbol Preferred_WUT:Yageo CC0402KRX7R8BB104 -> AAA_Preferred_WUT:Yageo CC0402KRX7R8BB104
- C75: renamed from C55; symbol Preferred_WUT:Yageo CC0402KRX7R8BB104 -> AAA_Preferred_WUT:Yageo CC0402KRX7R8BB104
- C76: renamed from C58; symbol Preferred_WUT:Yageo CC0402KRX7R8BB104 -> AAA_Preferred_WUT:Yageo CC0402KRX7R8BB104
- C77: renamed from C61; symbol Preferred_WUT:Yageo CC0402KRX7R8BB104 -> AAA_Preferred_WUT:Yageo CC0402KRX7R8BB104
- C82: renamed from C62; symbol Preferred_WUT:Yageo CC0402KRX7R8BB104 -> AAA_Preferred_WUT:Yageo CC0402KRX7R8BB104
- C84, C90, C91: renamed from C7; symbol Preferred_WUT:Samsung Electro-Mechanics CL10A106MO8NQNC -> AAA_Preferred_WUT:Samsung Electro-Mechanics CL10A106MO8NQNC
- C87: renamed from C64; symbol Preferred_WUT:Yageo CC0402KRX7R8BB104 -> AAA_Preferred_WUT:Yageo CC0402KRX7R8BB104
- C92: renamed from C26; symbol Preferred_WUT:Yageo CC0402KRX7R8BB104 -> AAA_Preferred_WUT:Yageo CC0402KRX7R8BB104
- C93: renamed from C3; symbol Preferred_WUT:Yageo CC0402KRX7R8BB104 -> AAA_Preferred_WUT:Yageo CC0402KRX7R8BB104
- C94: renamed from C29; symbol Preferred_WUT:Yageo CC0402KRX7R8BB104 -> AAA_Preferred_WUT:Yageo CC0402KRX7R8BB104
- C95: renamed from C32; symbol Preferred_WUT:Yageo CC0402KRX7R8BB104 -> AAA_Preferred_WUT:Yageo CC0402KRX7R8BB104
- C96: renamed from C111; symbol Preferred_WUT:Yageo CC0402KRX7R8BB104 -> AAA_Preferred_WUT:Yageo CC0402KRX7R8BB104
- C97: renamed from C114; symbol Preferred_WUT:Yageo CC0402KRX7R8BB104 -> AAA_Preferred_WUT:Yageo CC0402KRX7R8BB104
- C98: renamed from C164; symbol Preferred_WUT:Yageo CC0402KRX7R8BB104 -> AAA_Preferred_WUT:Yageo CC0402KRX7R8BB104
- C99: renamed from C165; symbol Preferred_WUT:Yageo CC0402KRX7R8BB104 -> AAA_Preferred_WUT:Yageo CC0402KRX7R8BB104
- FB12: renamed from FB8; symbol Preferred_WUT:Murata BLM15BD182SN1D -> AAA_Preferred_WUT:Murata BLM15BD182SN1D
- FB13: renamed from FB9; symbol Preferred_WUT:Murata BLM15BD182SN1D -> AAA_Preferred_WUT:Murata BLM15BD182SN1D
- FB14: renamed from FB10; symbol Preferred_WUT:Murata BLM15BD182SN1D -> AAA_Preferred_WUT:Murata BLM15BD182SN1D
- FB15: renamed from FB11; symbol Preferred_WUT:Murata BLM15BD182SN1D -> AAA_Preferred_WUT:Murata BLM15BD182SN1D
- FB16: renamed from FB12; symbol Preferred_WUT:Murata BLM15BD182SN1D -> AAA_Preferred_WUT:Murata BLM15BD182SN1D
- FB17: renamed from FB13; symbol Preferred_WUT:Murata BLM15BD182SN1D -> AAA_Preferred_WUT:Murata BLM15BD182SN1D
- FB18: renamed from FB14; symbol Preferred_WUT:Murata BLM18AG601SN1D -> AAA_Preferred_WUT:Murata BLM18AG601SN1D
- FB19: renamed from FB28; symbol Preferred_WUT:Murata BLM18AG601SN1D -> AAA_Preferred_WUT:Murata BLM18AG601SN1D
- FB20: renamed from FB15; symbol Preferred_WUT:Murata BLM15BD182SN1D -> AAA_Preferred_WUT:Murata BLM15BD182SN1D
- R85: renamed from R29; symbol Preferred_WUT:KOA Speer RK73H1ETTP1000F -> AAA_Preferred_WUT:KOA Speer RK73H1ETTP1000F
- renumbered C37 to C64, C42 to C65, C46 to C66, C50 to C67, C54 to C68, C57 to C69, C60 to C70, C22 to C78, C44 to C79, C48 to C80, C52 to C81, C69 to C83, C63 to C85, C67 to C86, C68 to C88, C151 to C89, R119 to R84, R121 to R86, T1 to T2, T2 to T3, T7 to T5, U4 to U13, U13 to U14

Commit message: less than 100 tracks to go!
Changed lines of the file:
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@@
     )
     (property "Voltage" "25V" (at 223.52 83.82 0) (do_not_autoplace)
-      (effects (font (size 1.27 1.27) (color 0 100 100 1)) (justify left))
+      (effects (font (size 1.27 1.27) (color 0 100 100 1)) (justify left) hide)
     )
     (property "Manufacturer" "Yageo" (at 220.98 86.36 0)
@@
     )
     (property "Voltage" "25V" (at 223.52 148.59 0) (do_not_autoplace)
-      (effects (font (size 1.27 1.27) (color 0 100 100 1)) (justify left))
+      (effects (font (size 1.27 1.27) (color 0 100 100 1)) (justify left) hide)
     )
     (property "Manufacturer" "Yageo" (at 220.98 151.13 0)
@@
     )
     (property "Voltage" "25V" (at 223.52 106.68 0) (do_not_autoplace)
-      (effects (font (size 1.27 1.27) (color 0 100 100 1)) (justify left))
+      (effects (font (size 1.27 1.27) (color 0 100 100 1)) (justify left) hide)
     )
     (property "Manufacturer" "Yageo" (at 220.98 109.22 0)
@@
     )
     (property "Voltage" "25V" (at 223.52 96.52 0) (do_not_autoplace)
-      (effects (font (size 1.27 1.27) (color 0 100 100 1)) (justify left))
+      (effects (font (size 1.27 1.27) (color 0 100 100 1)) (justify left) hide)
     )
     (property "Manufacturer" "Yageo" (at 220.98 99.06 0)
@@
     )
     (property "Voltage" "25V" (at 223.52 138.43 0) (do_not_autoplace)
-      (effects (font (size 1.27 1.27) (color 0 100 100 1)) (justify left))
+      (effects (font (size 1.27 1.27) (color 0 100 100 1)) (justify left) hide)
     )
     (property "Manufacturer" "Yageo" (at 220.98 140.97 0)
@@
     )
     (property "Voltage" "25V" (at 223.52 73.66 0) (do_not_autoplace)
-      (effects (font (size 1.27 1.27) (color 0 100 100 1)) (justify left))
+      (effects (font (size 1.27 1.27) (color 0 100 100 1)) (justify left) hide)
     )
     (property "Manufacturer" "Yageo" (at 220.98 76.2 0)
@@
     )
     (property "Voltage" "25V" (at 223.52 118.11 0) (do_not_autoplace)
-      (effects (font (size 1.27 1.27) (color 0 100 100 1)) (justify left))
+      (effects (font (size 1.27 1.27) (color 0 100 100 1)) (justify left) hide)
     )
     (property "Manufacturer" "Yageo" (at 220.98 120.65 0)
@@
     )
     (property "Voltage" "25V" (at 223.52 128.27 0) (do_not_autoplace)
-      (effects (font (size 1.27 1.27) (color 0 100 100 1)) (justify left))
+      (effects (font (size 1.27 1.27) (color 0 100 100 1)) (justify left) hide)
     )
     (property "Manufacturer" "Yageo" (at 220.98 130.81 0)

Commit message: committing before attempting scripting
Parts:
- renumbered C99 to C100, C57 to C58, C58 to C59, C59 to C60, C60 to C61, C61 to C62, C62 to C63, C63 to C64, C64 to C65, C65 to C66, C66 to C67, C67 to C68, C68 to C69, C69 to C70, C70 to C71, C71 to C72, C72 to C73, C73 to C74, C74 to C75, C75 to C76, C76 to C77, C77 to C78, C78 to C79, C79 to C80, C80 to C81, C81 to C82, C82 to C83, C83 to C84, C84 to C85, C85 to C86, C86 to C87, C87 to C88, C88 to C89, C89 to C90, C90 to C91, C91 to C92, C92 to C93, C93 to C94, C94 to C95, C95 to C96, C96 to C97, C97 to C98, C98 to C99, R84 to R86, R85 to R87, R86 to R88
