File: gps.kicad_sch (KiCad schematic)
At the start: 69 parts, among them CN1 CONSMA002-L-G, Q10 MMBT2907A-7-F, Q7 DMN62D0U-7, Q9 MMBT2907A-7-F, U16 SN74LVC2G157DCU, U17 ZED-F9T-10B, U18 TLV7031DCK, U3 TI TPS79301DBV, U4 TI TPS79301DBV, U7 SN74LVC1G125DBV

Commit message: stuff
Parts:
- added C14, C4: 47p, Capacitor_SMD:C_0402_1005Metric, symbol Auto_Library_WUT:Kemet C0402C470F5GACTU
- added FL3: B39162B8389P810, RF_WUT:Qualcomm_B8389, symbol RF_WUT:Qualcomm_B39162B8389P810
- added L7, L8: 5n1, Inductor_SMD:L_0402_1005Metric, symbol Auto_Library_WUT:Coilcraft 0402DC-5N1XJRW
Connections:
- net 0V: now also FL3.2, FL3.3, FL3.5, L7.2, L8.2
- net at CN1.1 (In), D20.1 (K), L1.2: now also C4.2; no longer U17.2 (RF_IN)
- net VCC_GNSS: now reaches C13.1, C15.1, C17.1, C20.1, C21.1, C39.1, R20.1, TP1.1, U17.33 (VCC), U17.34 (VCC), U17.36 (V_BCKP), U3.6 (OUT)
- new net: C14.1, FL3.1 (IN), L8.1
- new net: C14.2, U17.2 (RF_IN)
- new net: C4.1, FL3.4 (OUT), L7.1
Other:
- moved on the sheet: C18, CN1, D20, L1, R109, R112, R123, R124, U18

Commit message: layout progress
Parts:
- removed R114: 10R, Resistor_SMD:R_0805_2012Metric, symbol Auto_Library_WUT:KOA Speer RK73H2ATTD10R0F
- added R79: 10R, Resistor_SMD:R_0402_1005Metric, symbol Auto_Library_WUT:KOA Speer RK73H1ETTP10R0F
- C31: renamed from C8; symbol Preferred_WUT:Samsung Electro-Mechanics CL10A106MO8NQNC -> AAA_Preferred_WUT:Samsung Electro-Mechanics CL10A106MO8NQNC
- C32: renamed from C7; symbol Preferred_WUT:Samsung Electro-Mechanics CL10A106MO8NQNC -> AAA_Preferred_WUT:Samsung Electro-Mechanics CL10A106MO8NQNC
- C33: renamed from C10; symbol Preferred_WUT:Yageo CC0402KRX7R8BB104 -> AAA_Preferred_WUT:Yageo CC0402KRX7R8BB104
- C34: renamed from C9; symbol Preferred_WUT:Yageo CC0402KRX7R8BB104 -> AAA_Preferred_WUT:Yageo CC0402KRX7R8BB104
- C35: renamed from C121; symbol Preferred_WUT:Yageo CC0402KRX7R8BB104 -> AAA_Preferred_WUT:Yageo CC0402KRX7R8BB104
- C36: renamed from C118; symbol Preferred_WUT:Yageo CC0402KRX7R8BB104 -> AAA_Preferred_WUT:Yageo CC0402KRX7R8BB104
- C37: renamed from C159; symbol Preferred_WUT:Yageo CC0402KRX7R8BB104 -> AAA_Preferred_WUT:Yageo CC0402KRX7R8BB104
- C40: renamed from C16; symbol Preferred_WUT:Samsung Electro-Mechanics CL10A106MO8NQNC -> AAA_Preferred_WUT:Samsung Electro-Mechanics CL10A106MO8NQNC
- C41: renamed from C15; symbol Preferred_WUT:Samsung Electro-Mechanics CL10A106MO8NQNC -> AAA_Preferred_WUT:Samsung Electro-Mechanics CL10A106MO8NQNC
- C42: renamed from C17; symbol Preferred_WUT:Samsung Electro-Mechanics CL10A106MO8NQNC -> AAA_Preferred_WUT:Samsung Electro-Mechanics CL10A106MO8NQNC
- C44: renamed from C144; symbol Preferred_WUT:Yageo CC0402KRX7R8BB104 -> AAA_Preferred_WUT:Yageo CC0402KRX7R8BB104
- C47: renamed from C19; symbol Preferred_WUT:Yageo CC0402KRX7R8BB104 -> AAA_Preferred_WUT:Yageo CC0402KRX7R8BB104
- C48: renamed from C169; symbol Preferred_WUT:Samsung Electro-Mechanics CL10A106MO8NQNC -> AAA_Preferred_WUT:Samsung Electro-Mechanics CL10A106MO8NQNC
- C49: renamed from C39; symbol Preferred_WUT:Yageo CC0402KRX7R8BB104 -> AAA_Preferred_WUT:Yageo CC0402KRX7R8BB104
- C50: renamed from C21; symbol Preferred_WUT:Yageo CC0402KRX7R8BB104 -> AAA_Preferred_WUT:Yageo CC0402KRX7R8BB104
- C51: renamed from C20; symbol Preferred_WUT:Yageo CC0402KRX7R8BB104 -> AAA_Preferred_WUT:Yageo CC0402KRX7R8BB104
- C52: renamed from C156; symbol Preferred_WUT:Yageo CC0402KRX7R8BB104 -> AAA_Preferred_WUT:Yageo CC0402KRX7R8BB104
- C55: renamed from C18; symbol Preferred_WUT:Yageo CC0402KRX7R8BB104 -> AAA_Preferred_WUT:Yageo CC0402KRX7R8BB104
- D19: renamed from D20; symbol Preferred_WUT:Littelfuse AQ3522-01LTG -> AAA_Preferred_WUT:Littelfuse AQ3522-01LTG
- FB10: renamed from FB2; symbol Preferred_WUT:Murata BLM15BD182SN1D -> AAA_Preferred_WUT:Murata BLM15BD182SN1D
- FB11: renamed from FB3; symbol Preferred_WUT:Murata BLM15BD182SN1D -> AAA_Preferred_WUT:Murata BLM15BD182SN1D
- FB4: renamed from FB30; symbol Preferred_WUT:Murata BLM15BD182SN1D -> AAA_Preferred_WUT:Murata BLM15BD182SN1D
- FB5: renamed from FB4; symbol Preferred_WUT:Murata BLM15BD182SN1D -> AAA_Preferred_WUT:Murata BLM15BD182SN1D
- FB6: renamed from FB24; symbol Preferred_WUT:Murata BLM15BD182SN1D -> AAA_Preferred_WUT:Murata BLM15BD182SN1D
- FB7: renamed from FB5; symbol Preferred_WUT:Murata BLM15BD182SN1D -> AAA_Preferred_WUT:Murata BLM15BD182SN1D
- FB8: renamed from FB31; symbol Preferred_WUT:Murata BLM15BD182SN1D -> AAA_Preferred_WUT:Murata BLM15BD182SN1D
- FB9: renamed from FB6; symbol Preferred_WUT:Murata BLM15BD182SN1D -> AAA_Preferred_WUT:Murata BLM15BD182SN1D
- LD6: renamed from LD5; symbol Preferred_WUT:Ekinglux_E6C0603VGAC1UDA -> AAA_Preferred_WUT:Ekinglux_E6C0603VGAC1UDA
- R64: renamed from R19; symbol Preferred_WUT:KOA Speer RK73H1ETTP33R0F -> AAA_Preferred_WUT:KOA Speer RK73H1ETTP33R0F
- R65: renamed from R133; symbol Preferred_WUT:KOA Speer RK73H1ETTP33R0F -> AAA_Preferred_WUT:KOA Speer RK73H1ETTP33R0F
- R66: renamed from R134; symbol Preferred_WUT:KOA Speer RK73H1ETTP33R0F -> AAA_Preferred_WUT:KOA Speer RK73H1ETTP33R0F
- R67: renamed from R16; symbol Preferred_WUT:KOA Speer RK73H1ETTP33R0F -> AAA_Preferred_WUT:KOA Speer RK73H1ETTP33R0F
- R72: renamed from R137; symbol Preferred_WUT:KOA Speer RK73H1ETTP1002F -> AAA_Preferred_WUT:KOA Speer RK73H1ETTP1002F
- R73: renamed from R17; symbol Preferred_WUT:KOA Speer RK73H1ETTP33R0F -> AAA_Preferred_WUT:KOA Speer RK73H1ETTP33R0F
- R75: renamed from R18; symbol Preferred_WUT:KOA Speer RK73H1ETTP33R0F -> AAA_Preferred_WUT:KOA Speer RK73H1ETTP33R0F
- R76: renamed from R125; symbol Preferred_WUT:KOA Speer RK73H1ETTP1002F -> AAA_Preferred_WUT:KOA Speer RK73H1ETTP1002F
- R77: renamed from R135; symbol Preferred_WUT:KOA Speer RK73H1ETTP33R0F -> AAA_Preferred_WUT:KOA Speer RK73H1ETTP33R0F
- R78: renamed from R113; symbol Preferred_WUT:KOA Speer RK73H1ETTP1001F -> AAA_Preferred_WUT:KOA Speer RK73H1ETTP1001F
- R80: renamed from R123; symbol Preferred_WUT:KOA Speer RK73H1ETTP1002F -> AAA_Preferred_WUT:KOA Speer RK73H1ETTP1002F
- R82: renamed from R109; symbol Preferred_WUT:KOA Speer RK73H1ETTP1000F -> AAA_Preferred_WUT:KOA Speer RK73H1ETTP1000F
- R83: renamed from R112; symbol Preferred_WUT:KOA Speer RK73H1ETTP1002F -> AAA_Preferred_WUT:KOA Speer RK73H1ETTP1002F
- renumbered C119 to C30, C11 to C38, C13 to C39, C12 to C43, C5 to C45, C6 to C46, C168 to C53, C14 to C54, C4 to C56, CN1 to CN12, FL3 to FL2, L8 to L3, L7 to L4, L1 to L5, Q7 to Q2, Q9 to Q3, Q10 to Q4, R22 to R68, R23 to R69, R20 to R70, R21 to R71, R84 to R74, R124 to R81, TP1 to TP3, TP5 to TP4, U16 to U10, U17 to U11, U18 to U12, U4 to U7, U3 to U8, U7 to U9
Connections:
- net at C48.1, FB9.1, Q3.2 (E): now also R79.1
- net at Q3.1 (B), Q4.2 (E): now also R79.2
Other:
- note added: "Current limit of roughly 70mA"

Commit message: committing before attempting scripting
Parts:
- renumbered C30 to C31, C31 to C32, C32 to C33, C33 to C34, C34 to C35, C35 to C36, C36 to C37, C37 to C38, C38 to C39, C39 to C40, C40 to C41, C41 to C42, C42 to C43, C43 to C44, C44 to C45, C45 to C46, C46 to C47, C47 to C48, C48 to C49, C49 to C50, C50 to C51, C51 to C52, C52 to C53, C53 to C54, C54 to C55, C55 to C56, C56 to C57, R64 to R66, R65 to R67, R66 to R68, R67 to R69, R68 to R70, R69 to R71, R70 to R72, R71 to R73, R72 to R74, R73 to R75, R74 to R76, R75 to R77, R76 to R78, R77 to R79, R78 to R80, R79 to R81, R80 to R82, R81 to R83, R82 to R84, R83 to R85

Commit message: Think complete - apart from 12V connection
Removed accidential step file
Parts:
- added CN14: M20-9990446, Connector_PinHeader_2.54mm:PinHeader_1x06_P2.54mm_Vertical, symbol Connector_WUT:Harwin_M20-9990646
Connections:
- net 0V: now also CN14.6 (Pin_2)
- net VCC_GNSS: now also CN14.1 (Pin_1)
- net at Q2.3 (D), U11.49 (~{RESET}): now also CN14.5 (Pin_2)
- net GNSS_CLK: now reaches R75.1, U10.1 (A)
- net at C46.1, FB10.2, U11.42 (TXD/SPI_MISO): now also CN14.4 (Pin_2)
- new net GPS_CLK: CN14.3 (Pin_2)
Other:
- note added: "Optional connector for alternative GPS receiver"
Changed lines of the file:
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@@
   (junction (at 81.28 48.26) (diameter 0) (color 0 0 0 0)
   )
+  (junction (at 215.9 129.54) (diameter 0) (color 0 0 0 0)
+  )
+  (junction (at 218.44 147.32) (diameter 0) (color 0 0 0 0)
+  )
   (junction (at 139.7 96.52) (diameter 0) (color 0 0 0 0)
   )
@@
   (junction (at 152.4 96.52) (diameter 0) (color 0 0 0 0)
   )
+  (junction (at 204.47 96.52) (diameter 0) (color 0 0 0 0)
+  )
   (junction (at 314.96 132.08) (diameter 0) (color 0 0 0 0)
   )
@@
     (stroke (width 0) (type default))
   )
+  (wire (pts (xy 208.28 73.66) (xy 224.79 73.66))
+    (stroke (width 0) (type default))
+  )
   (wire (pts (xy 285.75 48.26) (xy 285.75 67.31))
     (stroke (width 0) (type default))
@@
     (stroke (width 0) (type default))
   )
-  (wire (pts (xy 238.76 147.32) (xy 209.55 147.32))
+  (wire (pts (xy 238.76 147.32) (xy 218.44 147.32))
     (stroke (width 0) (type default))
   )
@@
     (stroke (width 0) (type default))
   )
+  (wire (pts (xy 215.9 76.2) (xy 224.79 76.2))
+    (stroke (width 0) (type default))
+  )
   (wire (pts (xy 115.57 58.42) (xy 115.57 62.23))
     (stroke (width 0) (type default))
@@
     (stroke (width 0) (type default))
   )
+  (wire (pts (xy 215.9 129.54) (xy 213.36 129.54))
+    (stroke (width 0) (type default))
+  )
   (wire (pts (xy 191.77 170.18) (xy 191.77 172.72))
     (stroke (width 0) (type default))
@@
     (stroke (width 0) (type default))
   )
-  (wire (pts (xy 238.76 129.54) (xy 213.36 129.54))
+  (wire (pts (xy 238.76 129.54) (xy 215.9 129.54))
     (stroke (width 0) (type default))
   )
@@
     (stroke (width 0) (type default))
   )
+  (wire (pts (xy 218.44 147.32) (xy 209.55 147.32))
+    (stroke (width 0) (type default))
+  )
   (wire (pts (xy 92.71 215.9) (xy 92.71 218.44))
     (stroke (width 0) (type default))
   )
+  (wire (pts (xy 218.44 147.32) (xy 218.44 78.74))
+    (stroke (width 0) (type default))
+  )
   (wire (pts (xy 337.82 43.18) (xy 349.25 43.18))
     (stroke (width 0) (type default))
@@
     (stroke (width 0) (type default))
   )
+  (wire (pts (xy 215.9 76.2) (xy 215.9 129.54))
+    (stroke (width 0) (type default))
+  )
   (wire (pts (xy 71.12 166.37) (xy 93.98 166.37))
     (stroke (width 0) (type default))
@@
     (stroke (width 0) (type default))
   )
-  (wire (pts (xy 152.4 96.52) (xy 226.06 96.52))
+  (wire (pts (xy 152.4 96.52) (xy 204.47 96.52))
     (stroke (width 0) (type default))
   )
@@
     (stroke (width 0) (type default))
   )
+  (wire (pts (xy 204.47 68.58) (xy 204.47 96.52))
+    (stroke (width 0) (type default))
+  )
   (wire (pts (xy 176.53 161.29) (xy 180.34 161.29))
     (stroke (width 0) (type default))
@@
     (stroke (width 0) (type default))
   )
+  (wire (pts (xy 204.47 96.52) (xy 226.06 96.52))
+    (stroke (width 0) (type default))
+  )
   (wire (pts (xy 152.4 106.68) (xy 152.4 109.22))
     (stroke (width 0) (type default))
@@
     (stroke (width 0) (type default))
   )
+  (wire (pts (xy 222.25 81.28) (xy 224.79 81.28))
+    (stroke (width 0) (type default))
+  )
   (wire (pts (xy 110.49 62.23) (xy 115.57 62.23))
     (stroke (width 0) (type default))
   )
+  (wire (pts (xy 224.79 68.58) (xy 204.47 68.58))
+    (stroke (width 0) (type default))
+  )
   (wire (pts (xy 356.87 132.08) (xy 361.95 132.08))
     (stroke (width 0) (type default))
@@
     (stroke (width 0) (type default))
   )
+  (wire (pts (xy 222.25 83.82) (xy 222.25 81.28))
+    (stroke (width 0) (type default))
+  )
   (wire (pts (xy 158.75 231.14) (xy 172.72 231.14))
     (stroke (width 0) (type default))
   )
+  (wire (pts (xy 218.44 78.74) (xy 224.79 78.74))
+    (stroke (width 0) (type default))
+  )
   (wire (pts (xy 314.96 132.08) (xy 317.5 132.08))
     (stroke (width 0) (type default))
@@
     (effects (font (size 1.27 1.27)) (justify left bottom))
   )
+  (text "Optional connector\nfor alternative\nGPS receiver" (at 219.71 66.04 0)
+    (effects (font (size 1.27 1.27)) (justify left bottom))
+  )
   (text "Current limit of roughly 70mA" (at 288.29 64.77 0)
     (effects (font (size 1.27 1.27)) (justify left bottom))
@@
     (effects (font (size 1.27 1.27)) (justify right bottom))
   )
+  (label "GNSS_CLK" (at 133.35 231.14 180) (fields_autoplaced)
+    (effects (font (size 1.27 1.27)) (justify right bottom))
+  )
+  (label "GPS_CLK" (at 208.28 73.66 0) (fields_autoplaced)
+    (effects (font (size 1.27 1.27)) (justify left bottom))
+  )
   (hierarchical_label "PTP_PPS" (shape output) (at 46.99 166.37 180) (fields_autoplaced)
     (effects (font (size 1.27 1.27)) (justify right))
@@
     )
   )
+  (symbol (lib_id "Power_WUT:0V") (at 222.25 83.82 0) (unit 1)
+    (in_bom no) (on_board no) (dnp no) (fields_autoplaced)
+    (property "Reference" "#PWR0301" (at 222.25 83.82 0)
+      (effects (font (size 1.27 1.27)) hide)
+    )
+    (property "Value" "0V" (at 222.25 86.36 0) (do_not_autoplace)
+      (effects (font (size 1.27 1.27)))
+    )
+    (property "Footprint" "" (at 222.25 83.82 0)
+      (effects (font (size 1.27 1.27)) hide)
+    )
+    (property "Datasheet" "" (at 222.25 83.82 0)
+      (effects (font (size 1.27 1.27)) hide)
+    )
+    (pin "1")
+    (instances
+      (project "Master Timing Card"
+        (path "/6e8e281e-e30f-459d-852f-231836068db5/231ba923-6354-4319-a55b-e8f523b1b9f4"
+          (reference "#PWR0301") (unit 1)
+        )
+      )
+    )
+  )
   (symbol (lib_id "Auto_Library_WUT:Kemet C0402C472K5RACTU ") (at 298.45 110.49 0) (unit 1)
     (in_bom yes) (on_board yes) (dnp no) (fields_autoplaced)
@@
   (symbol (lib_id "RF_WUT:Qualcomm_B39162B8389P810") (at 327.66 132.08 0) (unit 1)
     (in_bom yes) (on_board yes) (dnp no)
-    (property "Reference" "FL2" (at 321.31 128.27 0) (do_not_autoplace)
+    (property "Reference" "FL2" (at 321.31 127 0) (do_not_autoplace)
       (effects (font (size 1.27 1.27)))
     )
-    (property "Value" "B39162B8389P810" (at 326.39 128.27 0) (do_not_autoplace)
+    (property "Value" "B39162B8389P810" (at 326.39 127 0) (do_not_autoplace)
       (effects (font (size 1.27 1.27)) (justify left))
     )
@@
         )
       )
+    )
+  )
+  (symbol (lib_id "Connector_WUT:Harwin_M20-9990646") (at 224.79 68.58 0) (unit 1)
+    (in_bom yes) (on_board yes) (dnp yes) (fields_autoplaced)
+    (property "Reference" "CN14" (at 231.14 73.66 0)
+      (effects (font (size 1.27 1.27)) (justify left))
+    )
+    (property "Value" "M20-9990446" (at 231.14 76.2 0)
+      (effects (font (size 1.27 1.27)) (justify left))
+    )
+    (property "Footprint" "Connector_PinHeader_2.54mm:PinHeader_1x06_P2.54mm_Vertical" (at 224.79 68.58 0)
+      (effects (font (size 1.27 1.27)) hide)
+    )
+    (property "Datasheet" "https://cdn.harwin.com/pdfs/M20-999.pdf" (at 224.79 68.58 0)
+      (effects (font (size 1.27 1.27)) hide)
+    )
+    (property "Manufacturer" "Harwin" (at 224.79 68.58 0)
+      (effects (font (size 1.27 1.27)) hide)
+    )
+    (property "MPN" "M20-9990646" (at 224.79 68.58 0)
+      (effects (font (size 1.27 1.27)) hide)
+    )
+    (pin "1")
+    (pin "3")
+    (pin "2")
+    (pin "4")
+    (pin "6")
+    (pin "5")
+    (instances
+      (project "Master Timing Card"
+        (path "/6e8e281e-e30f-459d-852f-231836068db5/231ba923-6354-4319-a55b-e8f523b1b9f4"
+          (reference "CN14") (unit 1)
+        )
+      )

Commit message: released version
Parts:
- removed C44: 100p, Capacitor_SMD:C_0402_1005Metric, symbol Auto_Library_WUT:Kemet C0402C101G5GACTU
- added C44: 22p, Capacitor_SMD:C_0402_1005Metric, symbol Auto_Library_WUT:Kemet C0402C220C5GACTU
Connections:
- net GPS_CLK is gone; now on net GNSS_CLK: CN14.3 (Pin_2)
- net 0V: now also C44.2
- net GNSS_CLK_M: now also C44.1
- net GNSS_PPS: now also CN14.2 (Pin_2)
- net GNSS_RX: now also C46.1, CN14.4 (Pin_2)
- net GNSS_TX: now also C47.1, CN14.5 (Pin_2)
- net at Q2.3 (D), U11.49 (~{RESET}): no longer CN14.5 (Pin_2)
- net at FB10.2, U11.42 (TXD/SPI_MISO): no longer C46.1, CN14.4 (Pin_2)
- net at FB11.2, U11.43 (RXD/SPI_MOSI): no longer C47.1
Other:
- moved on the sheet: C46, C47, FB10, FB11, R69, R77
