File: gps.kicad_sch (KiCad schematic)
At the start: 75 parts, among them CN12 CONSMA002-L-G, CN14 M20-9990446, Q2 DMN62D0U-7, Q3 MMBT2907A-7-F, Q4 MMBT2907A-7-F, U10 SN74LVC2G157DCU, U11 ZED-F9T-10B, U12 TLV7031DCK, U7 TI TPS79301DBV, U8 TI TPS79301DBV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

Commit message: .
Parts:
- U12: MPN (none) -> TLV7031DCK; Manufacturer (none) -> Texas Instruments
Changed lines of the file:
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@@
+			)
+		)
+		(property "Manufacturer" "Texas Instruments"
+			(at 349.25 72.39 0)
+			(effects
+				(font
+					(size 1.27 1.27)
+				)
+				(hide yes)
+			)
+		)
+		(property "MPN" "TLV7031DCK"
+			(at 349.25 72.39 0)
+			(effects
+				(font
+					(size 1.27 1.27)
+				)
+				(hide yes)
 			)
 		)
