File: cm4_hpio.kicad_sch (KiCad schematic)
At the start: 22 parts, among them CN5 USB4110-GF-A, CN7 TE 1-2199230-6, CN8 M2 x 2.5mm

Commit message: .
Parts:
- D13: value USBLC6-2M6 -> USBULC6-2M6; symbol Diode_WUT:USBLC6-2M6 -> Diode_WUT:USBULC6-2M6; MPN (none) -> USBULC6-2M6; Manufacturer (none) -> ST Microelectronics
Changed lines of the file:
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@@
 	)
 	(symbol
-		(lib_id "Diode_WUT:USBLC6-2M6")
+		(lib_id "Diode_WUT:USBULC6-2M6")
 		(at 76.2 191.77 0)
 		(unit 1)
@@
 			)
 		)
-		(property "Value" "USBLC6-2M6"
+		(property "Value" "USBULC6-2M6"
 			(at 83.82 196.85 0)
 			(effects
@@
 			(at 76.2 191.77 0)
 			(effects
+				(font
+					(size 1.27 1.27)
+				)
+				(hide yes)
+			)
+		)
+		(property "Manufacturer" "ST Microelectronics"
+			(at 76.2 191.77 0)
+			(effects
+				(font
+					(size 1.27 1.27)
+				)
+				(hide yes)
+			)
+		)
+		(property "MPN" "USBULC6-2M6"
+			(at 76.2 191.77 0)
+			(effects
